Commit message: Velodyne is floating

File: vehicle_autonomy/propbot_description/urdf/accessories/VLP-16.urdf.xacro (robot description, xacro)
@@ -27,11 +27,12 @@
 <robot xmlns:xacro="http://www.ros.org/wiki/xacro" name="VLP-16">
   <xacro:property name="M_PI" value="3.1415926535897931" />
-  <xacro:macro name="VLP-16" params="*origin parent:=base_link name:=velodyne topic:=/velodyne_points hz:=10 lasers:=16 samples:=1875 collision_range:=0.3 min_range:=0.9 max_range:=130.0 noise:=0.008 min_angle:=-${M_PI} max_angle:=${M_PI} gpu:=false frame:=base_laser">
+  <xacro:macro name="VLP-16" params="*origin parent:=base_laser_mount name:=base_laser topic:=/velodyne_points hz:=10 lasers:=16 samples:=1875 collision_range:=0.3 min_range:=0.9 max_range:=130.0 noise:=0.008 min_angle:=-${M_PI} max_angle:=${M_PI} gpu:=false">
     <joint name="${name}_mount_joint" type="fixed">
       <xacro:insert_block name="origin" />
       <parent link="${parent}"/>
-      <child link="${name}_base_link"/>
+      <child link="${name}_shell"/>
     </joint>
-    <link name="${name}_base_link">
+    <!-- Link to Velodyne Puck. -->
+    <link name="${name}_shell">
       <inertial>
         <mass value="0.83"/>
@@ -60,7 +61,8 @@
     <joint name="${name}_scan_joint" type="fixed" >
       <origin xyz="0 0 0.0377" rpy="0 0 0" />
-      <parent link="${name}_base_link" />
+      <parent link="${name}_shell" />
       <child link="${name}"/>
     </joint>
+    <!-- Link to sensor -->
     <link name="${name}">
       <inertial>
@@ -111,5 +113,5 @@
           <plugin name="gazebo_ros_laser_controller" filename="libgazebo_ros_velodyne_gpu_laser.so">
             <topicName>${topic}</topicName>
-            <frameName>${frame}</frameName>
+            <frameName>${name}</frameName>
             <min_range>${min_range}</min_range>
             <max_range>${max_range}</max_range>
@@ -151,5 +153,5 @@
           <plugin name="gazebo_ros_laser_controller" filename="libgazebo_ros_velodyne_laser.so">
             <topicName>${topic}</topicName>
-            <frameName>${frame}</frameName>
+            <frameName>${name}</frameName>
             <min_range>${min_range}</min_range>
             <max_range>${max_range}</max_range>

File: vehicle_autonomy/propbot_description/urdf/accessories/VLP-16_mount.urdf.xacro (robot description, xacro)
@@ -45,5 +45,5 @@
     </link>
       <!-- This offset is from the base of the bracket to the LIDAR's focal point. -->
-     <VLP-16 name="velodyne" frame="base_laser" topic="scan" hz="10" samples="440" parent="${prefix}_laser_mount">
+     <VLP-16 name="base_laser" topic="camera/depth/points" hz="10" samples="440" parent="${prefix}_laser_mount">
       <origin xyz="0 0 0.4" rpy="0 0 0" />
      </VLP-16>

File: vehicle_autonomy/propbot_description/urdf/propbot.urdf.xacro (robot description, xacro)
@@ -23,6 +23,6 @@
 <robot name="propbot" xmlns:xacro="http://ros.org/wiki/xacro">
   <xacro:arg name="laser_enabled" default="false" />
-  <xacro:arg name="laser_xyz" default="$(optenv PROPBOT_LMS1XX_XYZ 0.2206 0.0 0.00635)" />
-  <xacro:arg name="laser_rpy" default="$(optenv PROPBOT_LMS1XX_RPY 0.0 0.0 0.0)" />
+  <xacro:arg name="laser_xyz" default="$(optenv PROPBOT_VLP-16_XYZ 0.2206 0.0 0.00635)" />
+  <xacro:arg name="laser_rpy" default="$(optenv PROPBOT_VLP-16_RPY 0.0 0.0 0.0)" />
   <xacro:arg name="kinect_enabled" default="false" />
   <xacro:arg name="kinect_xyz" default="$(optenv PROPBOT_KINECT_XYZ 0 0 0)" />

Commit message: removed unnecessary mesh files

File: vehicle_autonomy/propbot_description/urdf/accessories/VLP-16.urdf.xacro (robot description, xacro)
@@ -44,10 +44,10 @@
       <visual>
         <geometry>
-          <mesh filename="package://propbot_description/meshes/VLP16_base_1.dae" />
+          <mesh filename="package://velodyne_description/meshes/VLP16_base_1.dae" />
         </geometry>
       </visual>
       <visual>
         <geometry>
-          <mesh filename="package://propbot_description/meshes/VLP16_base_2.dae" />
+          <mesh filename="package://velodyne_description/meshes/VLP16_base_2.dae" />
         </geometry>
       </visual>
@@ -74,5 +74,5 @@
         <origin xyz="0 0 -0.0377" />
         <geometry>
-          <mesh filename="package://propbot_description/meshes/VLP16_scan.dae" />
+          <mesh filename="package://velodyne_description/meshes/VLP16_scan.dae" />
         </geometry>
       </visual>

File: vehicle_autonomy/propbot_description/urdf/accessories/VLP-16_mount.urdf.xacro (robot description, xacro)
@@ -46,5 +46,5 @@
       <!-- This offset is from the base of the bracket to the LIDAR's focal point. -->
      <VLP-16 name="base_laser" topic="camera/depth/points" hz="10" samples="440" parent="${prefix}_laser_mount">
-      <origin xyz="0.0352 0 1" rpy="0 0 0" />
+      <origin xyz="0.0352 0 0.11" rpy="0 0 0" />
      </VLP-16>
   </xacro:macro>
