Commit message: fixed some errors introduced by cherry picking

File: vehicle_autonomy/propbot_description/urdf/accessories/realsense_d435.urdf.xacro (robot description, xacro)
@@ -102,5 +102,5 @@
           </clip>
         </camera>
-        <plugin name="kinect_${name}_controller" filename="libgazebo_ros_openni_kinect.so">
+        <plugin name="realsense_${name}_controller" filename="libgazebo_ros_openni_kinect.so">
           <cameraName>${name}</cameraName>
           <alwaysOn>true</alwaysOn>

File: vehicle_autonomy/propbot_description/urdf/propbot.urdf.xacro (robot description, xacro)
@@ -36,5 +36,5 @@
   <xacro:include filename="$(find propbot_description)/urdf/decorations.urdf.xacro" />
   <xacro:include filename="$(find propbot_description)/urdf/wheel.urdf.xacro" />
-  <xacro:include filename="$(find propbot_description)/urdf/accessories/kinect_camera.urdf.xacro"/>
+  <xacro:include filename="$(find propbot_description)/urdf/accessories/realsense_d435.urdf.xacro"/>
   <xacro:include filename="$(find propbot_description)/urdf/accessories/sensor_arch.urdf.xacro"/>
   <xacro:include filename="$(find propbot_description)/urdf/accessories/VLP-16_mount.urdf.xacro"/>
@@ -128,6 +128,6 @@
       <origin xyz="-0.35 0 0.51" rpy="0 0 -3.14"/>
     </xacro:sensor_arch>
-    <joint name="kinect_frame_joint" type="fixed">
-      <origin xyz="$(arg kinect_xyz)" rpy="$(arg kinect_rpy)" />
+    <joint name="rgbd_camera_frame_joint" type="fixed">
+      <origin xyz="$(arg rgbd_camera_xyz)" rpy="$(arg rgbd_camera_rpy)" />
       <parent link="sensor_arch_mount_link"/>
       <child link="camera_link"/>

Commit message: removed some unnecessary urdf parameters, added comment for realsense FOV

File: vehicle_autonomy/propbot_description/urdf/accessories/realsense_d435.urdf.xacro (robot description, xacro)
@@ -30,9 +30,4 @@
   <xacro:macro name="realsense_d435" params="parent *origin name:=camera robot_namespace:=/">
     <xacro:property name="M_PI" value="3.1415926535897931" />
-    <!-- The following values are approximate, and the camera node
-     publishing TF values with actual calibrated camera extrinsic values -->
-    <xacro:property name="d435_cam_depth_to_infra1_offset" value="0.0"/>
-    <xacro:property name="d435_cam_depth_to_infra2_offset" value="-0.050"/>
-    <xacro:property name="d435_cam_depth_to_color_offset" value="0.015"/>
     <!-- The following values model the aluminum peripherial case for the
   	D435 camera, with the camera joint represented by the actual
@@ -91,4 +86,5 @@
         <update_rate>20.0</update_rate>
         <camera>
+          <!-- Horizontal FOV is 69 degrees -->
           <horizontal_fov>${69.0*M_PI/180.0}</horizontal_fov>
           <image>

Commit message: added ground removal fitlers, filter for velodyne still needs tuning

File: vehicle_autonomy/propbot_description/urdf/accessories/realsense_d435.urdf.xacro (robot description, xacro)
@@ -86,6 +86,6 @@
         <update_rate>20.0</update_rate>
         <camera>
-          <!-- Horizontal FOV is 69 degrees -->
-          <horizontal_fov>${69.0*M_PI/180.0}</horizontal_fov>
+          <!-- Horizontal FOV is 55 degrees (actual FOV is 69 deg)-->
+          <horizontal_fov>${55.0*M_PI/180.0}</horizontal_fov>
           <image>
             <format>R8G8B8</format>

File: vehicle_autonomy/propbot_description/urdf/propbot.urdf.xacro (robot description, xacro)
@@ -128,9 +128,4 @@
       <origin xyz="-0.35 0 0.51" rpy="0 0 -3.14"/>
     </xacro:sensor_arch>
-    <joint name="rgbd_camera_frame_joint" type="fixed">
-      <origin xyz="$(arg rgbd_camera_xyz)" rpy="$(arg rgbd_camera_rpy)" />
-      <parent link="sensor_arch_mount_link"/>
-      <child link="camera_link"/>
-    </joint>
     <realsense_d435 name="camera" parent="sensor_arch_mount_link">
       <origin xyz="$(arg rgbd_camera_xyz)" rpy="$(arg rgbd_camera_rpy)" robot_namespace="$(arg robot_namespace)"/>
