Commit message: #99 Update URDF files to work with Propbot STL files and test in simulation  (#166)
* Replaces husky model with propbot model

Co-authored-by: Divya Budihal <divyabudihal@gmail.com>

File: vehicle_autonomy/propbot_description/urdf/propbot.urdf.xacro (robot description, xacro)
@@ -21,55 +21,133 @@
 ARISING IN ANY WAY OUT OF THE USE OF THIS SOFTWARE, EVEN IF ADVISED OF THE POSSIBILITY OF SUCH DAMAGE.
 -->
+<!-- NOTES
+* All values are in metric (m, kg)
+* Specific robot structure values extracted from URDF exported from Solidworks
+-->
 <robot name="propbot" xmlns:xacro="http://ros.org/wiki/xacro">
-  <xacro:arg name="laser_enabled" default="false" />
-  <xacro:arg name="laser_xyz" default="$(optenv PROPBOT_VLP-16_XYZ 0.2206 0.0 0.00635)" />
-  <xacro:arg name="laser_rpy" default="$(optenv PROPBOT_VLP-16_RPY 0.0 0.0 0.0)" />
-  <xacro:arg name="rgbd_camera_enabled" default="false" />
-  <xacro:arg name="rgbd_camera_xyz" default="$(optenv PROPBOT_REALSENSE_XYZ 0 0 0)" />
-  <xacro:arg name="rgbd_camera_rpy" default="$(optenv PROPBOT_REALSENSE_RPY 0 0.18 3.14)" />
-  <xacro:property name="propbot_front_bumper_extend" value="$(optenv PROPBOT_FRONT_BUMPER_EXTEND 0)" />
-  <xacro:property name="propbot_rear_bumper_extend" value="$(optenv PROPBOT_REAR_BUMPER_EXTEND 0)" />
+  <!--
+  ***********************************************************************************************
+  Default Spawn Settings
+  ***********************************************************************************************
+  -->
   <xacro:arg name="robot_namespace" default="/" />
   <xacro:arg name="spawn_lat" default="49.9" />
   <xacro:arg name="spawn_long" default="8.9" />
-  <!-- Included URDF/XACRO Files -->
+  <!--
+  ***********************************************************************************************
+  Base Size Specifications
+  ***********************************************************************************************
+  The "shadow" of the robot
+  -->
+  <xacro:property name="base_x_size" value="0.9820" /> <!-- x is front to back -->
+  <xacro:property name="base_y_size" value="0.8278" /> <!-- y is side to side -->
+  <xacro:property name="base_z_size" value="0.1369" /> <!-- height of the bottom battery plate from the ground -->
+  <!--
+  ***********************************************************************************************
+  Misc. Constants
+  ***********************************************************************************************
+  -->
+  <xacro:property name="M_PI" value="3.14159"/>
+  <!--
+  ***********************************************************************************************
+  Laser and Camera Args
+  ***********************************************************************************************
+  -->
+  <xacro:arg name="laser_enabled" default="false" />
+  <xacro:arg name="laser_xyz" default="$(optenv PROPBOT_VLP-16_XYZ 0.08 ${-base_y_size/2 + 0.0516/2} 0.925)" /> <!-- note: base_y_size/2 + lidar radius -->
+  <xacro:arg name="laser_rpy" default="$(optenv PROPBOT_VLP-16_RPY 0 0 0)" />
+  <xacro:arg name="rgbd_camera_enabled" default="false" />
+  <xacro:arg name="rgbd_camera_xyz" default="$(optenv PROPBOT_REALSENSE_XYZ 0 0 0.225)" />
+  <xacro:arg name="rgbd_camera_rpy" default="$(optenv PROPBOT_REALSENSE_RPY 0 0.18 0)" />
+  <!--
+  ***********************************************************************************************
+  Included URDF/XACRO Files
+  ***********************************************************************************************
+  -->
   <xacro:include filename="$(find propbot_description)/urdf/decorations.urdf.xacro" />
   <xacro:include filename="$(find propbot_description)/urdf/wheel.urdf.xacro" />
+  <xacro:include filename="$(find propbot_description)/urdf/passive_wheel.urdf.xacro" />
   <xacro:include filename="$(find propbot_description)/urdf/accessories/realsense_d435.urdf.xacro"/>
   <xacro:include filename="$(find propbot_description)/urdf/accessories/sensor_arch.urdf.xacro"/>
   <xacro:include filename="$(find propbot_description)/urdf/accessories/VLP-16_mount.urdf.xacro"/>
-  <xacro:property name="M_PI" value="3.14159"/>
-  <!-- Base Size -->
-  <xacro:property name="base_x_size" value="0.98740000" />
-  <xacro:property name="base_y_size" value="0.57090000" />
-  <xacro:property name="base_z_size" value="0.24750000" />
+  <!--
+  ***********************************************************************************************
+  Mass and Inertial Values and Scaling
+  ***********************************************************************************************
+  Values as reported by SolidWorks
+  -->
+  <!-- Approximate REAL robot mass -->
+  <xacro:property name="robot_mass" value="70.0"/>
+  <!-- SW reported mass values -->
+  <xacro:property name="base_link_mass" value="0.96268" />
+  <xacro:property name="chassis_mass" value="19.52246"/>
+  <xacro:property name="wheel_mass" value="2.96542"/>
+  <!-- Base link inertia-->
+  <xacro:property name="base_ixx" value="0.083320" />
+  <xacro:property name="base_ixy" value="-1.882647E-14" />
+  <xacro:property name="base_ixz" value="2.527076E-19" />
+  <xacro:property name="base_iyy" value="0.003905" />
+  <xacro:property name="base_iyz" value="7.039418E-19" />
+  <xacro:property name="base_izz" value="0.087218" />
+   <!-- Chassis link inertia-->
+  <xacro:property name="chassis_ixx" value="0.42226" />
+  <xacro:property name="chassis_ixy" value="0.00028" />
+  <xacro:property name="chassis_ixz" value="-0.00012" />
+  <xacro:property name="chassis_iyy" value="0.46973" />
+  <xacro:property name="chassis_iyz" value="0.00017" />
+  <xacro:property name="chassis_izz" value="0.16238" />
+  <!-- Robot frame mass scale factor: use to scale chassis and base link masses and inertial values -->
+  <xacro:property name="frame_msf" value="${robot_mass/chassis_mass}" />
+  <!-- Wheel mass scale factor: use to scale wheel masses and inertial values -->
+  <xacro:property name="wheel_msf" value="1" />
+  <!--
+  ***********************************************************************************************
+  Wheel Properties and Mounting Specifications
+  ***********************************************************************************************
+  -->
+  <!-- Wheel Properties -->
+  <xacro:property name="wheel_length" value="0.08975" />
+  <xacro:property name="wheel_radius" value="0.127" />
   <!-- Wheel Mounting Positions -->
-  <xacro:property name="wheelbase" value="0.5120" />
-  <xacro:property name="track" value="0.5708" />
-  <xacro:property name="wheel_vertical_offset" value="0.03282" />
-  <!-- Wheel Properties -->
-  <xacro:property name="wheel_length" value="0.1143" />
-  <xacro:property name="wheel_radius" value="0.1651" />
+  <xacro:property name="wheel_to_wheel" value="0.400" /> <!-- distance between wheel axles -->
+  <xacro:property name="track" value="0.9198" /> <!-- y wheel distance, wheel central point to central point -->
+  <xacro:property name="wheel_vertical_offset" value="${wheel_radius}" /> <!-- axle to ground distance -->
+  <xacro:property name="wheel_central_offset" value="0.0533" /> <!-- offset from the center -->
+  <!--
+  ***********************************************************************************************
+  Sensor Mounting Specifications
+  ***********************************************************************************************
+  -->
+  <xacro:property name="top_plate_height" value="${0.24845 + wheel_radius}" /> <!-- height from the ground to the top plate -->
+  <xacro:property name="top_plate_front" value="${base_x_size/2}" /> <!-- distance from the origin to the front of the robot -->
+  <!--
+  ***********************************************************************************************
+  Linking and Joint Specification
+  ***********************************************************************************************
+  The various links and joints are created and put together
+  -->
+  <!--
+  Base Link
+  ======================================================================
+  -->
   <!-- Base link is the center of the robot's bottom plate -->
   <link name="base_link">
     <visual>
-      <origin xyz="0 0 0" rpy="0 0 0" />
+      <origin xyz="0 0 ${base_z_size}" rpy="0 0 ${-M_PI/2}" />
       <geometry>
-        <mesh filename="package://propbot_description/meshes/base_link.dae" />
+        <mesh filename="package://propbot_description/meshes/propbot_base_link.STL" />
       </geometry>
     </visual>
     <collision>
-      <origin xyz="${( propbot_front_bumper_extend - propbot_rear_bumper_extend ) / 2.0} 0 ${base_z_size/4}" rpy="0 0 0" />
+      <origin xyz="0 ${wheel_central_offset + wheel_length/2} ${base_z_size/4}" rpy="0 0 ${-M_PI/2}" />
       <geometry>
-        <box size="${ base_x_size + propbot_front_bumper_extend + propbot_rear_bumper_extend } ${base_y_size} ${base_z_size/2}"/>
-      </geometry>
-    </collision>
-    <collision>
-      <origin xyz="0 0 ${base_z_size*3/4-0.01}" rpy="0 0 0" />
-      <geometry>
-        <box size="${base_x_size*4/5} ${base_y_size} ${base_z_size/2-0.02}"/>
+        <box size="${base_x_size} ${base_y_size} ${base_z_size/2}"/>
       </geometry>
     </collision>
   </link>
+  <!-- Set base_link colour in Gazebo -->
+  <gazebo reference="base_link">
+    <material>Gazebo/Red</material>
+  </gazebo>
   <!-- Base footprint is on the ground under the robot -->
   <link name="base_footprint"/>
@@ -79,10 +157,21 @@
     <child link="base_footprint" />
   </joint>
-  <!-- Interial link stores the robot's inertial information -->
+  <!--
+  Inertial Link
+  ======================================================================
+  Interial link stores the robot's inertial information
+  For this case, the mass, origin, and inertia values of the main chassis is used
+  -->
   <link name="inertial_link">
     <inertial>
-      <mass value="46.034" />
-      <origin xyz="-0.00065 -0.085 0.062" />
-      <inertia ixx="0.6022" ixy="-0.02364" ixz="-0.1197" iyy="1.7386" iyz="-0.001544" izz="2.0296" />
+      <mass value="${(chassis_mass + base_link_mass) * frame_msf}"/>
+      <origin xyz="-0.004962 0.10679 0.42243" rpy = "${-M_PI/2} ${-M_PI/2} 0" />
+      <inertia
+        ixx="${(base_ixx + chassis_ixx) * frame_msf}"
+        ixy="${(base_ixy + chassis_ixy) * frame_msf}"
+        ixz="${(base_ixz + chassis_ixz) * frame_msf}"
+        iyy="${(base_iyy + chassis_iyy) * frame_msf}"
+        iyz="${(base_iyz + chassis_iyz) * frame_msf}"
+        izz="${(base_izz + chassis_izz) * frame_msf}" />
     </inertial>
   </link>
@@ -92,6 +181,10 @@
     <child link="inertial_link" />
   </joint>
-  <!-- IMU Link is the standard mounting position for the UM6 IMU.-->
-  <!-- Can be modified with environment variables in /etc/ros/setup.bash -->
+  <!--
+  IMU Link
+  ======================================================================
+  IMU Link is the standard mounting position for the UM6 IMU.
+  Can be modified with environment variables in /etc/ros/setup.bash
+  -->
   <link name="imu_link"/>
   <joint name="imu_joint" type="fixed">
@@ -102,18 +195,35 @@
   <gazebo reference="imu_link">
   </gazebo>
-  <!-- Propbot wheel macros -->
+  <!--
+  Wheels
+  ======================================================================
+  -->
+  <!-- Right -->
+  <xacro:propbot_wheel wheel_prefix="front_right">
+    <origin xyz="${track/2} ${-wheel_to_wheel} ${wheel_vertical_offset}" rpy="0 0 ${-M_PI/2}" />
+  </xacro:propbot_wheel>
+  <xacro:propbot_wheel wheel_prefix="rear_right">
+    <origin xyz="${-track/2 + (2/3)*wheel_radius} ${-wheel_to_wheel} ${wheel_vertical_offset}" rpy="0 0 ${-M_PI/2}" />
+  </xacro:propbot_wheel>
+  <!-- Left -->
   <xacro:propbot_wheel wheel_prefix="front_left">
-    <origin xyz="${wheelbase/2} ${track/2} ${wheel_vertical_offset}" rpy="0 0 0" />
-  </xacro:propbot_wheel>
-  <xacro:propbot_wheel wheel_prefix="front_right">
-    <origin xyz="${wheelbase/2} ${-track/2} ${wheel_vertical_offset}" rpy="0 0 0" />
+    <origin xyz="${track/2} ${wheel_to_wheel} ${wheel_vertical_offset}" rpy="0 0 ${-M_PI/2}" />
   </xacro:propbot_wheel>
   <xacro:propbot_wheel wheel_prefix="rear_left">
-    <origin xyz="${-wheelbase/2} ${track/2} ${wheel_vertical_offset}" rpy="0 0 0" />
-  </xacro:propbot_wheel>
-  <xacro:propbot_wheel wheel_prefix="rear_right">
-    <origin xyz="${-wheelbase/2} ${-track/2} ${wheel_vertical_offset}" rpy="0 0 0" />
-  </xacro:propbot_wheel>
+    <origin xyz="${-track/2 + (2/3)*wheel_radius} ${wheel_to_wheel} ${wheel_vertical_offset}" rpy="0 0 ${-M_PI/2}" />
+  </xacro:propbot_wheel>
+  <!-- Middle (passives) -->
+  <xacro:propbot_passive_wheel wheel_prefix="left">
+    <origin xyz="${wheel_radius/3} ${wheel_to_wheel} ${wheel_vertical_offset}" rpy="0 0 ${-M_PI/2}" />
+  </xacro:propbot_passive_wheel>
+  <xacro:propbot_passive_wheel wheel_prefix="right">
+    <origin xyz="${wheel_radius/3} ${-wheel_to_wheel} ${wheel_vertical_offset}" rpy="0 0 ${-M_PI/2}" />
+  </xacro:propbot_passive_wheel>
+  <!-- Decorate the robot -->
   <xacro:propbot_decorate />
+  <!--
+  Laser and Camera
+  ======================================================================
+  -->
   <xacro:if value="$(arg laser_enabled)">
     <VLP-16_mount prefix="base" />
@@ -126,5 +236,5 @@
   <xacro:if value="$(arg rgbd_camera_enabled)">
     <xacro:sensor_arch prefix="" parent="top_plate_link">
-      <origin xyz="-0.35 0 0.51" rpy="0 0 -3.14"/>
+      <origin xyz="${base_x_size/2 - 0.05} ${-base_y_size/2 + 0.025} 0.6" rpy="0 0 0"/>
     </xacro:sensor_arch>
     <realsense_d435 name="camera" parent="sensor_arch_mount_link">
@@ -132,4 +242,10 @@
      </realsense_d435>
   </xacro:if>
+  <!--
+  ***********************************************************************************************
+  Gazebo Specifications
+  ***********************************************************************************************
+  -->
+  <!-- Motion controller -->
   <gazebo>
     <plugin name="gazebo_ros_control" filename="libgazebo_ros_control.so">
@@ -137,4 +253,5 @@
     </plugin>
   </gazebo>
+  <!-- IMU controller -->
   <gazebo>
     <plugin name="imu_controller" filename="libhector_gazebo_ros_imu.so">
@@ -151,4 +268,5 @@
     </plugin>
   </gazebo>
+  <!-- GPS controller -->
   <gazebo>
     <plugin name="gps_controller" filename="libhector_gazebo_ros_gps.so">

File: vehicle_autonomy/propbot_description/urdf/wheel.urdf.xacro (robot description, xacro)
@@ -24,14 +24,19 @@
 	<xacro:macro name="propbot_wheel" params="wheel_prefix *joint_pose">
 		<link name="${wheel_prefix}_wheel_link">
+			<!-- Following values extracted from URDF exported from Solidworks -->
 			<inertial>
-				<mass value="2.637" />
+				<mass value="${wheel_mass * wheel_msf}" />
 				<origin xyz="0 0 0" />
-				<inertia  ixx="0.02467" ixy="0" ixz="0" iyy="0.04411" iyz="0" izz="0.02467" />
+				<inertia  ixx="${0.01875 * wheel_msf}" ixy="${1.054410E-15 * wheel_msf}" ixz="${6.83081E-07 * wheel_msf}"
+				          iyy="${0.01012 * wheel_msf}" iyz="${-4.64239E-08 * wheel_msf}" izz="${0.01012 * wheel_msf}" />
 			</inertial>
 			<visual>
 				<origin xyz="0 0 0" rpy="0 0 0" />
 				<geometry>
-					<mesh filename="package://propbot_description/meshes/wheel.dae" />
+					<mesh filename="package://propbot_description/meshes/propbot_wheel.STL" />>
 				</geometry>
+				<material name="wheel_material">
+				  <color rgba="0.109804 0.109804 0.109804 1" />
+      			</material>
 			</visual>
 			<collision>
@@ -43,9 +48,10 @@
 		</link>
 		<gazebo reference="${wheel_prefix}_wheel_link">
-			<mu1 value="1.0"/>
-			<mu2 value="1.0"/>
+			<mu1 value="100.0"/>
+			<mu2 value="100.0"/>
 			<kp value="10000000.0" />
 			<kd value="1.0" />
 			<fdir1 value="1 0 0"/>
+      		<material>Gazebo/Black</material>
 		</gazebo>
 		<joint name="${wheel_prefix}_wheel" type="continuous">
@@ -53,5 +59,5 @@
 			<child link="${wheel_prefix}_wheel_link"/>
 			<xacro:insert_block name="joint_pose"/>
-			<axis xyz="0 1 0" rpy="0 0 0" />
+			<axis xyz="-1 0 0" rpy="0 0 0" />
 		</joint>
 		<transmission name="${wheel_prefix}_wheel_trans" type="SimpleTransmission">
