Commit message: Extra costmaps not removed, currently recognizes floor as obstacle

File: vehicle_autonomy/propbot_description/urdf/accessories/VLP-16_mount.urdf.xacro (robot description, xacro)
@@ -46,5 +46,5 @@
       <!-- This offset is from the base of the bracket to the LIDAR's focal point. -->
      <VLP-16 name="base_laser" topic="camera/depth/points" hz="10" samples="440" parent="${prefix}_laser_mount">
-      <origin xyz="0 0 0.4" rpy="0 0 0" />
+      <origin xyz="0.0352 0 1" rpy="0 0 0" />
      </VLP-16>
   </xacro:macro>

Commit message: LiDAR positioning fix

File: vehicle_autonomy/propbot_description/urdf/accessories/VLP-16_mount.urdf.xacro (robot description, xacro)
@@ -38,7 +38,7 @@
       </visual>
       <collision>
-        <origin xyz="0 0 .0585" rpy="0 0 0" />
+        <origin xyz="0 0 0.0585" rpy="0 0 0" />
         <geometry>
-          <box size=".1 .108 .117" />
+          <box size="0.1 0.108 0.117" />
         </geometry>
       </collision>
@@ -46,5 +46,5 @@
       <!-- This offset is from the base of the bracket to the LIDAR's focal point. -->
      <VLP-16 name="base_laser" topic="velodyne/points" hz="10" samples="440" parent="${prefix}_laser_mount" gpu="false">
-      <origin xyz="0.0352 0 0.11" rpy="0 0 0" />
+      <origin xyz="0.017 0 0.105" rpy="0 0 0" />
      </VLP-16>
   </xacro:macro>

File: vehicle_autonomy/propbot_description/urdf/decorations.urdf.xacro (robot description, xacro)
@@ -57,24 +57,22 @@
     A tiny plate use to link the sensors to the robot
     -->
-    <xacro:if value="$(optenv PROPBOT_TOP_PLATE_ENABLED true)">
-      <!-- Spawn the top plate -->
-      <link name="top_plate_link">
-        <visual>
-          <origin xyz="${base_x_size/2} ${-base_y_size/2 + 0.027} ${top_plate_height}" rpy="0 0 0" />
-          <geometry>
-            <box size="0.01 0.01 0.001"/>
-          </geometry>
-          <material name="wheel_material">
-				    <color rgba="0.25 0.25 0.75 0" />
-      		</material>
-        </visual>
-      </link>
-      <!-- Attach top plate to chassis -->
-      <joint name="top_plate_chassis_joint" type="fixed">
-        <parent link="chassis_link" />
-        <child link="top_plate_link"/>
-        <origin xyz="0 ${top_plate_front - base_y_size/8} 0.001" rpy="0 0 0"/>
-      </joint>
-    </xacro:if>
+    <!-- Spawn the top plate -->
+    <link name="top_plate_link">
+      <visual>
+        <origin xyz="${base_x_size/2} ${-base_y_size/2 + 0.027} ${top_plate_height}" rpy="0 0 0" />
+        <geometry>
+          <box size="0.01 0.01 0.001"/>
+        </geometry>
+        <material name="wheel_material">
+          <color rgba="0.25 0.25 0.75 0" />
+        </material>
+      </visual>
+    </link>
+    <!-- Attach top plate to chassis -->
+    <joint name="top_plate_chassis_joint" type="fixed">
+      <parent link="chassis_link" />
+      <child link="top_plate_link"/>
+      <origin xyz="0 ${top_plate_front - base_y_size/8} 0.001" rpy="0 0 0"/>
+    </joint>
   </xacro:macro>
 </robot>

File: vehicle_autonomy/propbot_description/urdf/propbot.urdf.xacro (robot description, xacro)
@@ -36,4 +36,13 @@
   <!--
   ***********************************************************************************************
+  Base Size Specifications
+  ***********************************************************************************************
+  The "shadow" of the robot
+  -->
+  <xacro:property name="base_x_size" value="0.9820" /> <!-- x is front to back -->
+  <xacro:property name="base_y_size" value="0.8278" /> <!-- y is side to side -->
+  <xacro:property name="base_z_size" value="0.1369" /> <!-- height of the bottom battery plate from the ground -->
+  <!--
+  ***********************************************************************************************
   Misc. Constants
   ***********************************************************************************************
@@ -46,8 +55,8 @@
   -->
   <xacro:arg name="laser_enabled" default="false" />
-  <xacro:arg name="laser_xyz" default="$(optenv PROPBOT_VLP-16_XYZ 0.2206 0.0 0.75)" />
-  <xacro:arg name="laser_rpy" default="$(optenv PROPBOT_VLP-16_RPY 0.0 0.0 0.0)" />
+  <xacro:arg name="laser_xyz" default="$(optenv PROPBOT_VLP-16_XYZ 0.02 ${-base_y_size/4 + 0.035} 0.925)" />
+  <xacro:arg name="laser_rpy" default="$(optenv PROPBOT_VLP-16_RPY 0 0 0)" />
   <xacro:arg name="rgbd_camera_enabled" default="false" />
-  <xacro:arg name="rgbd_camera_xyz" default="$(optenv PROPBOT_REALSENSE_XYZ 0 0 0)" />
+  <xacro:arg name="rgbd_camera_xyz" default="$(optenv PROPBOT_REALSENSE_XYZ 0 0 0.95)" />
   <xacro:arg name="rgbd_camera_rpy" default="$(optenv PROPBOT_REALSENSE_RPY 0 0.18 3.14)" />
   <!--
@@ -107,13 +116,4 @@
   <!--
   ***********************************************************************************************
-  Base Size Specifications
-  ***********************************************************************************************
-  The "shadow" of the robot
-  -->
-  <xacro:property name="base_x_size" value="0.9820" /> <!-- x is front to back -->
-  <xacro:property name="base_y_size" value="0.8278" /> <!-- y is side to side -->
-  <xacro:property name="base_z_size" value="0.1369" /> <!-- height of the bottom battery plate from the ground -->
-  <!--
-  ***********************************************************************************************
   Sensor Mounting Specifications
   ***********************************************************************************************

Commit message: Application of the lidar patch, simplified some  inertial components to 0

File: vehicle_autonomy/propbot_description/urdf/accessories/VLP-16_mount.urdf.xacro (robot description, xacro)
@@ -45,5 +45,5 @@
     </link>
       <!-- This offset is from the base of the bracket to the LIDAR's focal point. -->
-     <VLP-16 name="base_laser" topic="velodyne/points" hz="10" samples="440" parent="${prefix}_laser_mount" gpu="false">
+     <VLP-16 name="base_laser" topic="velodyne/points" hz="10" samples="440" parent="${prefix}_laser_mount" gpu="true">
       <origin xyz="0.017 0 0.105" rpy="0 0 0" />
      </VLP-16>

File: vehicle_autonomy/propbot_description/urdf/propbot.urdf.xacro (robot description, xacro)
@@ -85,15 +85,15 @@
   <!-- Base link inertia-->
   <xacro:property name="base_ixx" value="0.083320" />
-  <xacro:property name="base_ixy" value="-1.882647E-14" />
-  <xacro:property name="base_ixz" value="2.527076E-19" />
+  <xacro:property name="base_ixy" value="0" />
+  <xacro:property name="base_ixz" value="0" />
   <xacro:property name="base_iyy" value="0.003905" />
-  <xacro:property name="base_iyz" value="7.039418E-19" />
+  <xacro:property name="base_iyz" value="0" />
   <xacro:property name="base_izz" value="0.087218" />
    <!-- Chassis link inertia-->
   <xacro:property name="chassis_ixx" value="0.42226" />
   <xacro:property name="chassis_ixy" value="0.00028" />
-  <xacro:property name="chassis_ixz" value="-0.00012" />
+  <xacro:property name="chassis_ixz" value="0" />
   <xacro:property name="chassis_iyy" value="0.46973" />
-  <xacro:property name="chassis_iyz" value="0.00017" />
+  <xacro:property name="chassis_iyz" value="0" />
   <xacro:property name="chassis_izz" value="0.16238" />
   <!-- Robot frame mass scale factor: use to scale chassis and base link masses and inertial values -->
