Commit message: WIP switch to Propbot, fixes to wheel positions

File: vehicle_autonomy/propbot_description/urdf/decorations.urdf.xacro (robot description, xacro)
@@ -23,165 +23,18 @@
 <robot name="propbot_decorations" xmlns:xacro="http://ros.org/wiki/xacro">
   <xacro:macro name="propbot_decorate">
-    <xacro:property name="propbot_front_bumper_extend" value="$(optenv PROPBOT_FRONT_BUMPER_EXTEND 0)" />
-    <xacro:property name="propbot_rear_bumper_extend" value="$(optenv PROPBOT_REAR_BUMPER_EXTEND 0)" />
     <!-- Spawn Propbot chassis -->
-    <link name="top_chassis_link">
+    <link name="chassis_link">
       <visual>
-        <origin xyz="0 0 0" rpy="0 0 0" />
+        <origin xyz="0 ${base_x_size/2} ${2*wheel_vertical_offset - base_z_size}" rpy="${M_PI/2} 0 0" />
         <geometry>
-          <mesh filename="package://propbot_description/meshes/top_chassis.dae" />
+          <mesh filename="package://propbot_description/meshes/propbot_chassis.STL" />
         </geometry>
       </visual>
     </link>
     <!-- Attach chassis to the robot -->
-    <joint name="top_chassis_joint" type="fixed">
+    <joint name="chassis_joint" type="fixed">
       <parent link="base_link" />
-      <child link="top_chassis_link" />
+      <child link="chassis_link" />
     </joint>
-    <xacro:if value="$(optenv PROPBOT_USER_RAIL_ENABLED true)">
-      <!-- Spawn user rails -->
-      <link name="user_rail_link">
-        <visual>
-          <geometry>
-            <mesh filename="package://propbot_description/meshes/user_rail.dae" />
-          </geometry>
-        </visual>
-      </link>
-      <!-- Attach user rails to base link -->
-      <joint name="user_rail" type="fixed">
-        <origin xyz="0.272 0 0.245" rpy="0 0 0" />
-        <parent link="base_link" />
-        <child link="user_rail_link" />
-      </joint>
-    </xacro:if>
-    <!-- Spawn front bumper link -->
-    <link name="front_bumper_link">
-      <visual>
-        <geometry>
-          <mesh filename="package://propbot_description/meshes/bumper.dae" />
-        </geometry>
-      </visual>
-    </link>
-    <!-- Attach front bumper -->
-    <joint name="front_bumper" type="fixed">
-      <origin xyz="${0.48 + propbot_front_bumper_extend} 0 0.091" rpy="0 0 0" />
-      <parent link="base_link" />
-      <child link="front_bumper_link" />
-    </joint>
-    <xacro:if value="${propbot_front_bumper_extend}">
-      <link name="front_bumper_extension_link">
-          <visual>
-              <geometry>
-                  <mesh filename="package://propbot_description/meshes/bumper_extension.dae" />
-              </geometry>
-          </visual>
-      </link>
-      <joint name="front_bumper_extension" type="fixed">
-        <origin xyz="${0.48 + propbot_front_bumper_extend} 0 0.091" rpy="0 0 0" />
-        <parent link="base_link" />
-        <child link="front_bumper_extension_link" />
-      </joint>
-    </xacro:if>
-    <!-- Spawn rear bumper link -->
-    <link name="rear_bumper_link">
-      <visual>
-        <geometry>
-          <mesh filename="package://propbot_description/meshes/bumper.dae" />
-        </geometry>
-      </visual>
-    </link>
-    <!-- Attach rear bumper -->
-    <joint name="rear_bumper" type="fixed">
-      <origin xyz="${-0.48 - propbot_rear_bumper_extend} 0 0.091" rpy="0 0 ${M_PI}" />
-      <parent link="base_link" />
-      <child link="rear_bumper_link" />
-    </joint>
-    <xacro:if value="${propbot_rear_bumper_extend}">
-      <link name="rear_bumper_extension_link">
-          <visual>
-              <geometry>
-                  <mesh filename="package://propbot_description/meshes/bumper_extension.dae" />
-              </geometry>
-          </visual>
-      </link>
-      <joint name="rear_bumper_extension" type="fixed">
-        <origin xyz="${-0.48 - propbot_rear_bumper_extend} 0 0.091" rpy="0 0 ${M_PI}" />
-        <parent link="base_link" />
-        <child link="rear_bumper_extension_link" />
-      </joint>
-    </xacro:if>
-    <xacro:if value="$(optenv PROPBOT_TOP_PLATE_ENABLED true)">
-      <!-- Spawn the top plate -->
-      <xacro:if value="$(optenv PROPBOT_LARGE_TOP_PLATE false)">
-        <link name="top_plate_link">
-          <visual>
-            <origin xyz="0 0 0" rpy="0 0 0" />
-            <geometry>
-              <mesh filename="package://propbot_description/meshes/large_top_plate.dae" />
-            </geometry>
-          </visual>
-          <collision>
-            <origin xyz="0 0 0" rpy="0 0 0"/>
-            <geometry>
-              <mesh filename="package://propbot_description/meshes/large_top_plate_collision.stl" />
-            </geometry>
-          </collision>
-        </link>
-        <!-- Attach top plate -->
-        <joint name="top_plate_joint" type="fixed">
-          <parent link="base_link" />
-          <child link="top_plate_link"/>
-          <origin xyz="0.0812 0 0.225" rpy="0 0 0"/>
-        </joint>
-        <!-- Top plate front link -->
-        <joint name="top_plate_front_joint" type="fixed">
-          <parent link="top_plate_link" />
-          <child link="top_plate_front_link"/>
-          <origin xyz="0.4125 0 0.00672" rpy="0 0 0"/>
-        </joint>
-        <!-- Top plate rear link-->
-        <joint name="top_plate_rear_joint" type="fixed">
-          <parent link="top_plate_link" />
-          <child link="top_plate_rear_link"/>
-          <origin xyz="-0.4125 0 0.00672" rpy="0 0 0"/>
-        </joint>
-      </xacro:if>
-      <xacro:unless value="$(optenv PROPBOT_LARGE_TOP_PLATE false)">
-        <link name="top_plate_link">
-          <visual>
-            <origin xyz="0 0 0" rpy="0 0 0" />
-            <geometry>
-              <mesh filename="package://propbot_description/meshes/top_plate.dae" />
-            </geometry>
-          </visual>
-          <collision>
-            <origin xyz="0 0 0" rpy="0 0 0"/>
-            <geometry>
-              <mesh filename="package://propbot_description/meshes/top_plate.stl" />
-            </geometry>
-          </collision>
-        </link>
-        <!-- Attach top plate -->
-        <joint name="top_plate_joint" type="fixed">
-          <parent link="base_link" />
-          <child link="top_plate_link"/>
-          <origin xyz="0.0812 0 0.245" rpy="0 0 0"/>
-        </joint>
-        <!-- Top plate front link -->
-        <joint name="top_plate_front_joint" type="fixed">
-          <parent link="top_plate_link" />
-          <child link="top_plate_front_link"/>
-          <origin xyz="0.36367 0 0.00639" rpy="0 0 0"/>
-        </joint>
-        <!-- Top plate rear link-->
-        <joint name="top_plate_rear_joint" type="fixed">
-          <parent link="top_plate_link" />
-          <child link="top_plate_rear_link"/>
-          <origin xyz="-0.36633 0 0.00639" rpy="0 0 0"/>
-        </joint>
-      </xacro:unless>
-      <link name="top_plate_front_link"/>
-      <link name="top_plate_rear_link"/>
-    </xacro:if>
   </xacro:macro>
 </robot>

File: vehicle_autonomy/propbot_description/urdf/propbot.urdf.xacro (robot description, xacro)
@@ -2,5 +2,5 @@
 <!--
 Software License Agreement (BSD)
-\file      propbot.urdf.xacro
+\file      propbot-model.urdf.xacro
 \authors   Paul Bovbel <pbovbel@clearpathrobotics.com>, Devon Ash <dash@clearpathrobotics.com>
 \copyright Copyright (c) 2015, Clearpath Robotics, Inc., All rights reserved.
@@ -21,4 +21,9 @@
 ARISING IN ANY WAY OUT OF THE USE OF THIS SOFTWARE, EVEN IF ADVISED OF THE POSSIBILITY OF SUCH DAMAGE.
 -->
+<!-- NOTES
+==============================================================================================================
+* All values are in metric (m, kg)
+* Specific robot structure values extracted from URDF exported from Solidworks
+-->
 <robot name="propbot" xmlns:xacro="http://ros.org/wiki/xacro">
   <xacro:arg name="laser_enabled" default="false" />
@@ -28,6 +33,4 @@
   <xacro:arg name="rgbd_camera_xyz" default="$(optenv PROPBOT_REALSENSE_XYZ 0 0 0)" />
   <xacro:arg name="rgbd_camera_rpy" default="$(optenv PROPBOT_REALSENSE_RPY 0 0.18 3.14)" />
-  <xacro:property name="propbot_front_bumper_extend" value="$(optenv PROPBOT_FRONT_BUMPER_EXTEND 0)" />
-  <xacro:property name="propbot_rear_bumper_extend" value="$(optenv PROPBOT_REAR_BUMPER_EXTEND 0)" />
   <xacro:arg name="robot_namespace" default="/" />
   <xacro:arg name="spawn_lat" default="49.9" />
@@ -39,28 +42,28 @@
   <xacro:include filename="$(find propbot_description)/urdf/accessories/sensor_arch.urdf.xacro"/>
   <xacro:include filename="$(find propbot_description)/urdf/accessories/VLP-16_mount.urdf.xacro"/>
+  <!-- Define Constant(s) -->
   <xacro:property name="M_PI" value="3.14159"/>
+  <!-- Wheel Properties -->
+  <xacro:property name="wheel_radius" value="0.127" />
+  <!-- Wheel Mounting Positions -->
+  <xacro:property name="wheel_to_wheel" value="0.400" /> <!-- distance between wheel axles -->
+  <xacro:property name="track" value="0.9198" /> <!-- y wheel distance, wheel central point to central point -->
+  <xacro:property name="wheel_vertical_offset" value="${wheel_radius}" /> <!-- axle to ground distance -->
   <!-- Base Size -->
-  <xacro:property name="base_x_size" value="0.98740000" />
-  <xacro:property name="base_y_size" value="0.57090000" />
-  <xacro:property name="base_z_size" value="0.24750000" />
-  <!-- Wheel Mounting Positions -->
-  <xacro:property name="wheelbase" value="0.5120" />
-  <xacro:property name="track" value="0.5708" />
-  <xacro:property name="wheel_vertical_offset" value="0.03282" />
-  <!-- Wheel Properties -->
-  <xacro:property name="wheel_length" value="0.1143" />
-  <xacro:property name="wheel_radius" value="0.1651" />
+  <xacro:property name="base_x_size" value="0.9820" /> <!-- x is front to back -->
+  <xacro:property name="base_y_size" value="0.8278" /> <!-- y is side to side -->
+  <xacro:property name="base_z_size" value="0.1369" /> <!-- height of the bottom battery plate from the ground -->
   <!-- Base link is the center of the robot's bottom plate -->
   <link name="base_link">
     <visual>
-      <origin xyz="0 0 0" rpy="0 0 0" />
+      <origin xyz="0 0 ${base_z_size}" rpy="0 0 0" />
       <geometry>
-        <mesh filename="package://propbot_description/meshes/base_link.dae" />
+        <mesh filename="package://propbot_description/meshes/propbot_base_link.STL" />
       </geometry>
     </visual>
     <collision>
-      <origin xyz="${( propbot_front_bumper_extend - propbot_rear_bumper_extend ) / 2.0} 0 ${base_z_size/4}" rpy="0 0 0" />
+      <origin xyz="0 0 ${base_z_size/4}" rpy="0 0 0" />
       <geometry>
-        <box size="${ base_x_size + propbot_front_bumper_extend + propbot_rear_bumper_extend } ${base_y_size} ${base_z_size/2}"/>
+        <box size="${base_x_size} ${base_y_size} ${base_z_size/2}"/>
       </geometry>
     </collision>
@@ -79,10 +82,12 @@
     <child link="base_footprint" />
   </joint>
-  <!-- Interial link stores the robot's inertial information -->
+  <!-- Interial link stores the robot's inertial information
+       For this case, the mass, origin, and inertia values of the main chassis is used
+  -->
   <link name="inertial_link">
     <inertial>
-      <mass value="46.034" />
-      <origin xyz="-0.00065 -0.085 0.062" />
-      <inertia ixx="0.6022" ixy="-0.02364" ixz="-0.1197" iyy="1.7386" iyz="-0.001544" izz="2.0296" />
+      <mass value="19.52246" />
+      <origin xyz="-0.004962 0.106799 0.42243" />
+      <inertia ixx="0.42226" ixy="0.00028" ixz="-0.00012" iyy="0.46973" iyz="0.000170" izz="0.16238" />
     </inertial>
   </link>
@@ -104,14 +109,20 @@
   <!-- Propbot wheel macros -->
   <xacro:propbot_wheel wheel_prefix="front_left">
-    <origin xyz="${wheelbase/2} ${track/2} ${wheel_vertical_offset}" rpy="0 0 0" />
+    <origin xyz="${track/2} ${wheel_to_wheel + wheel_radius/4 + 0.011} ${wheel_vertical_offset}" rpy="0 ${M_PI} 0" />
   </xacro:propbot_wheel>
   <xacro:propbot_wheel wheel_prefix="front_right">
-    <origin xyz="${wheelbase/2} ${-track/2} ${wheel_vertical_offset}" rpy="0 0 0" />
+    <origin xyz="${-track/2} ${wheel_to_wheel} ${wheel_vertical_offset}" rpy="0 0 0" />
+  </xacro:propbot_wheel>
+  <xacro:propbot_wheel wheel_prefix="middle_left">
+    <origin xyz="${track/2} 0 ${wheel_vertical_offset}" rpy="0 ${M_PI} 0" />
+  </xacro:propbot_wheel>
+  <xacro:propbot_wheel wheel_prefix="middle_right">
+    <origin xyz="${-track/2} 0 ${wheel_vertical_offset}" rpy="0 0 0" />
   </xacro:propbot_wheel>
   <xacro:propbot_wheel wheel_prefix="rear_left">
-    <origin xyz="${-wheelbase/2} ${track/2} ${wheel_vertical_offset}" rpy="0 0 0" />
+    <origin xyz="${track/2} ${-wheel_to_wheel} ${wheel_vertical_offset}" rpy="0 ${M_PI} 0" />
   </xacro:propbot_wheel>
   <xacro:propbot_wheel wheel_prefix="rear_right">
-    <origin xyz="${-wheelbase/2} ${-track/2} ${wheel_vertical_offset}" rpy="0 0 0" />
+    <origin xyz="${-track/2} ${-wheel_to_wheel} ${wheel_vertical_offset}" rpy="0 0 0" />
   </xacro:propbot_wheel>
   <xacro:propbot_decorate />

File: vehicle_autonomy/propbot_description/urdf/wheel.urdf.xacro (robot description, xacro)
@@ -24,19 +24,23 @@
 	<xacro:macro name="propbot_wheel" params="wheel_prefix *joint_pose">
 		<link name="${wheel_prefix}_wheel_link">
+			<!-- Following values extracted from URDF exported from Solidworks -->
 			<inertial>
-				<mass value="2.637" />
+				<mass value="2.96542" />
 				<origin xyz="0 0 0" />
-				<inertia  ixx="0.02467" ixy="0" ixz="0" iyy="0.04411" iyz="0" izz="0.02467" />
+				<inertia  ixx="0.01875" ixy="1.054410E-15" ixz="6.83081E-07" iyy="0.01012" iyz="-4.64239E-08" izz="0.01012" />
 			</inertial>
 			<visual>
 				<origin xyz="0 0 0" rpy="0 0 0" />
 				<geometry>
-					<mesh filename="package://propbot_description/meshes/wheel.dae" />
+					<mesh filename="package://propbot_description/meshes/propbot_wheel.STL" />>
 				</geometry>
+				<material name="wheel_material">
+				  <color rgba="0.109804 0.109804 0.109804 1" />
+      			</material>
 			</visual>
 			<collision>
 				<origin xyz="0 0 0" rpy="${M_PI/2} 0 0" />
 				<geometry>
-					<cylinder length="${wheel_length}" radius="${wheel_radius}" />
+					<mesh filename="package://propbot_description/meshes/propbot_wheel.STL" />
 				</geometry>
 			</collision>
@@ -53,5 +57,5 @@
 			<child link="${wheel_prefix}_wheel_link"/>
 			<xacro:insert_block name="joint_pose"/>
-			<axis xyz="0 1 0" rpy="0 0 0" />
+			<axis xyz="1 0 0" rpy="0 0 0" />
 		</joint>
 		<transmission name="${wheel_prefix}_wheel_trans" type="SimpleTransmission">

Commit message: Fixes to the wheel positions

File: vehicle_autonomy/propbot_description/urdf/decorations.urdf.xacro (robot description, xacro)
@@ -26,5 +26,5 @@
     <link name="chassis_link">
       <visual>
-        <origin xyz="0 0 0" rpy="0 0 0" />
+        <origin xyz="0 ${base_x_size/2} ${2*wheel_vertical_offset - base_z_size}" rpy="${M_PI/2} 0 0" />
         <geometry>
           <mesh filename="package://propbot_description/meshes/propbot_chassis.STL" />

File: vehicle_autonomy/propbot_description/urdf/propbot.urdf.xacro (robot description, xacro)
@@ -21,5 +21,9 @@
 ARISING IN ANY WAY OUT OF THE USE OF THIS SOFTWARE, EVEN IF ADVISED OF THE POSSIBILITY OF SUCH DAMAGE.
 -->
-<!-- NOTE: all values are metric -->
+<!-- NOTES
+==============================================================================================================
+* All values are in metric (m, kg)
+* Specific robot structure values extracted from URDF exported from Solidworks
+-->
 <robot name="propbot" xmlns:xacro="http://ros.org/wiki/xacro">
   <xacro:arg name="laser_enabled" default="false" />
@@ -38,19 +42,20 @@
   <xacro:include filename="$(find propbot_description)/urdf/accessories/sensor_arch.urdf.xacro"/>
   <xacro:include filename="$(find propbot_description)/urdf/accessories/VLP-16_mount.urdf.xacro"/>
+  <!-- Define Constant(s) -->
   <xacro:property name="M_PI" value="3.14159"/>
   <!-- Wheel Properties -->
   <xacro:property name="wheel_radius" value="0.127" />
+  <!-- Wheel Mounting Positions -->
+  <xacro:property name="wheel_to_wheel" value="0.400" /> <!-- distance between wheel axles -->
+  <xacro:property name="track" value="0.9198" /> <!-- y wheel distance, wheel central point to central point -->
+  <xacro:property name="wheel_vertical_offset" value="${wheel_radius}" /> <!-- axle to ground distance -->
   <!-- Base Size -->
   <xacro:property name="base_x_size" value="0.9820" /> <!-- x is front to back -->
   <xacro:property name="base_y_size" value="0.8278" /> <!-- y is side to side -->
   <xacro:property name="base_z_size" value="0.1369" /> <!-- height of the bottom battery plate from the ground -->
-  <!-- Wheel Mounting Positions -->
-  <xacro:property name="wheel_to_wheel" value="0.400" /> <!-- distance between wheel axles -->
-  <xacro:property name="track" value="0.9198" /> <!-- y wheel distance, wheel central point to central point -->
-  <xacro:property name="wheel_vertical_offset" value="${wheel_radius}" /> <!-- axle to ground distance -->
   <!-- Base link is the center of the robot's bottom plate -->
   <link name="base_link">
     <visual>
-      <origin xyz="0 0 0" rpy="0 0 0" />
+      <origin xyz="0 0 ${base_z_size}" rpy="0 0 0" />
       <geometry>
         <mesh filename="package://propbot_description/meshes/propbot_base_link.STL" />
@@ -77,10 +82,12 @@
     <child link="base_footprint" />
   </joint>
-  <!-- Interial link stores the robot's inertial information -->
+  <!-- Interial link stores the robot's inertial information
+       For this case, the mass, origin, and inertia values of the main chassis is used
+  -->
   <link name="inertial_link">
     <inertial>
-      <mass value="46.034" />
-      <origin xyz="-0.00065 -0.085 0.062" />
-      <inertia ixx="0.6022" ixy="-0.02364" ixz="-0.1197" iyy="1.7386" iyz="-0.001544" izz="2.0296" />
+      <mass value="19.52246" />
+      <origin xyz="-0.004962 0.106799 0.42243" />
+      <inertia ixx="0.42226" ixy="0.00028" ixz="-0.00012" iyy="0.46973" iyz="0.000170" izz="0.16238" />
     </inertial>
   </link>
@@ -102,20 +109,20 @@
   <!-- Propbot wheel macros -->
   <xacro:propbot_wheel wheel_prefix="front_left">
-    <origin xyz="${wheel_to_wheel} ${track/2} ${wheel_vertical_offset}" rpy="0 0 0" />
+    <origin xyz="${track/2} ${wheel_to_wheel + wheel_radius/4 + 0.011} ${wheel_vertical_offset}" rpy="0 ${M_PI} 0" />
   </xacro:propbot_wheel>
   <xacro:propbot_wheel wheel_prefix="front_right">
-    <origin xyz="${wheel_to_wheel} ${-track/2} ${wheel_vertical_offset}" rpy="0 0 0" />
+    <origin xyz="${-track/2} ${wheel_to_wheel} ${wheel_vertical_offset}" rpy="0 0 0" />
   </xacro:propbot_wheel>
   <xacro:propbot_wheel wheel_prefix="middle_left">
-    <origin xyz="0 ${track/2} ${wheel_vertical_offset}" rpy="0 0 0" />
+    <origin xyz="${track/2} 0 ${wheel_vertical_offset}" rpy="0 ${M_PI} 0" />
   </xacro:propbot_wheel>
   <xacro:propbot_wheel wheel_prefix="middle_right">
-    <origin xyz="0 ${-track/2} ${wheel_vertical_offset}" rpy="0 0 0" />
+    <origin xyz="${-track/2} 0 ${wheel_vertical_offset}" rpy="0 0 0" />
   </xacro:propbot_wheel>
   <xacro:propbot_wheel wheel_prefix="rear_left">
-    <origin xyz="${-wheel_to_wheel} ${track/2} ${wheel_vertical_offset}" rpy="0 0 0" />
+    <origin xyz="${track/2} ${-wheel_to_wheel} ${wheel_vertical_offset}" rpy="0 ${M_PI} 0" />
   </xacro:propbot_wheel>
   <xacro:propbot_wheel wheel_prefix="rear_right">
-    <origin xyz="${-wheel_to_wheel} ${-track/2} ${wheel_vertical_offset}" rpy="0 0 0" />
+    <origin xyz="${-track/2} ${-wheel_to_wheel} ${wheel_vertical_offset}" rpy="0 0 0" />
   </xacro:propbot_wheel>
   <xacro:propbot_decorate />

File: vehicle_autonomy/propbot_description/urdf/wheel.urdf.xacro (robot description, xacro)
@@ -24,21 +24,23 @@
 	<xacro:macro name="propbot_wheel" params="wheel_prefix *joint_pose">
 		<link name="${wheel_prefix}_wheel_link">
+			<!-- Following values extracted from URDF exported from Solidworks -->
 			<inertial>
 				<mass value="2.96542" />
 				<origin xyz="0 0 0" />
-				<inertia
-				  ixx="0.01875" ixy="1.054410E-15" ixz="6.83081E-07"
-				  iyy="0.01012" iyz="-4.64239E-08" izz="0.01012" />
+				<inertia  ixx="0.01875" ixy="1.054410E-15" ixz="6.83081E-07" iyy="0.01012" iyz="-4.64239E-08" izz="0.01012" />
 			</inertial>
 			<visual>
 				<origin xyz="0 0 0" rpy="0 0 0" />
 				<geometry>
-					<mesh filename="package://propbot_model/meshes/propbot_wheel.STL" />>
+					<mesh filename="package://propbot_description/meshes/propbot_wheel.STL" />>
 				</geometry>
+				<material name="wheel_material">
+				  <color rgba="0.109804 0.109804 0.109804 1" />
+      			</material>
 			</visual>
 			<collision>
 				<origin xyz="0 0 0" rpy="${M_PI/2} 0 0" />
 				<geometry>
-					<mesh filename="package://propbot_model/meshes/propbot_wheel.STL" />
+					<mesh filename="package://propbot_description/meshes/propbot_wheel.STL" />
 				</geometry>
 			</collision>
@@ -55,5 +57,5 @@
 			<child link="${wheel_prefix}_wheel_link"/>
 			<xacro:insert_block name="joint_pose"/>
-			<axis xyz="0 1 0" rpy="0 0 0" />
+			<axis xyz="1 0 0" rpy="0 0 0" />
 		</joint>
 		<transmission name="${wheel_prefix}_wheel_trans" type="SimpleTransmission">
