Commit message: Added invisible top plate for sensor linking

File: vehicle_autonomy/propbot_description/urdf/decorations.urdf.xacro (robot description, xacro)
@@ -37,4 +37,24 @@
       <child link="chassis_link" />
     </joint>
+    <xacro:if value="$(optenv PROPBOT_TOP_PLATE_ENABLED true)">
+      <!-- Spawn "invisible" the top plate -->
+      <link name="top_plate_link">
+        <visual>
+          <origin xyz="0 0 ${top_plate_height}" rpy="0 0 0" />
+          <geometry>
+            <box size="0.001 0.001 0.001"/>
+          </geometry>
+          <material name="wheel_material">
+				    <color rgba="0.25 0.25 0.75 0" />
+      		</material>
+        </visual>
+      </link>
+      <!-- Attach top plate to chassis -->
+      <joint name="top_plate_chassis_joint" type="fixed">
+        <parent link="chassis_link" />
+        <child link="top_plate_link"/>
+        <origin xyz="0 ${top_plate_front - base_y_size/8} 0.001" rpy="0 0 0"/>
+      </joint>
+    </xacro:if>
   </xacro:macro>
 </robot>

File: vehicle_autonomy/propbot_description/urdf/propbot.urdf.xacro (robot description, xacro)
@@ -2,5 +2,5 @@
 <!--
 Software License Agreement (BSD)
-\file      propbot-model.urdf.xacro
+\file      propbot.urdf.xacro
 \authors   Paul Bovbel <pbovbel@clearpathrobotics.com>, Devon Ash <dash@clearpathrobotics.com>
 \copyright Copyright (c) 2015, Clearpath Robotics, Inc., All rights reserved.
@@ -55,4 +55,7 @@
   <xacro:property name="base_y_size" value="0.8278" /> <!-- y is side to side -->
   <xacro:property name="base_z_size" value="0.1369" /> <!-- height of the bottom battery plate from the ground -->
+  <!-- Sensor Mounting Values -->
+  <xacro:property name="top_plate_height" value="${0.24845 + wheel_radius}" /> <!-- height from the ground to the top plate-->
+  <xacro:property name="top_plate_front" value="${base_x_size/2}" /> <!-- distance from the origin to the front of the robot-->
   <!-- Base link is the center of the robot's bottom plate -->
   <link name="base_link">
@@ -138,5 +141,5 @@
   <xacro:if value="$(arg rgbd_camera_enabled)">
     <xacro:sensor_arch prefix="" parent="top_plate_link">
-      <origin xyz="-0.35 0 0.51" rpy="0 0 -3.14"/>
+      <origin xyz="0 0 0" rpy="0 0 -${M_PI}"/>
     </xacro:sensor_arch>
     <joint name="rgbd_camera_frame_joint" type="fixed">

File: vehicle_autonomy/propbot_description/urdf/propbot_model.urdf (robot description, URDF)
Before this commit: robot propbot_model, 9 links, 8 joints
Links:
- link base_link: geometry collision mesh filename=package://propbot_description/meshes/propbot_base_link.STL; visual mesh filename=package://propbot_description/meshes/propbot_base_link.STL
- link base_link_to_main_frame: geometry collision mesh filename=package://propbot_description/meshes/propbot_chassis.STL; visual mesh filename=package://propbot_description/meshes/propbot_chassis.STL
- link base_to_left_back_wheel: geometry collision mesh filename=package://propbot_description/meshes/propbot_wheel.STL; visual mesh filename=package://propbot_description/meshes/propbot_wheel.STL
- link base_to_left_front_wheel: geometry collision mesh filename=package://propbot_description/meshes/propbot_wheel.STL; visual mesh filename=package://propbot_description/meshes/propbot_wheel.STL
- link base_to_left_middle_wheel: geometry collision mesh filename=package://propbot_description/meshes/propbot_wheel.STL; visual mesh filename=package://propbot_description/meshes/propbot_wheel.STL
- link base_to_right_back_wheel: geometry collision mesh filename=package://propbot_description/meshes/propbot_wheel.STL; visual mesh filename=package://propbot_description/meshes/propbot_wheel.STL
- link base_to_right_front_wheel: geometry collision mesh filename=package://propbot_description/meshes/propbot_wheel.STL; visual mesh filename=package://propbot_description/meshes/propbot_wheel.STL
- link base_to_right_middle_wheel: geometry collision mesh filename=package://propbot_description/meshes/propbot_wheel.STL; visual mesh filename=package://propbot_description/meshes/propbot_wheel.STL

Commit message: Added in Gazebo material specifications for chassis and wheels

File: vehicle_autonomy/propbot_description/urdf/decorations.urdf.xacro (robot description, xacro)
@@ -32,4 +32,8 @@
       </visual>
     </link>
+    <!-- Set chassis colour in Gazebo -->
+    <gazebo reference="chassis_link">
+      <material>Gazebo/Red</material>
+    </gazebo>
     <!-- Attach chassis to the robot -->
     <joint name="chassis_joint" type="fixed">

File: vehicle_autonomy/propbot_description/urdf/propbot.urdf.xacro (robot description, xacro)
@@ -86,4 +86,8 @@
     </collision>
   </link>
+  <!-- Set base_link colour in Gazebo -->
+  <gazebo reference="base_link">
+    <material>Gazebo/Red</material>
+  </gazebo>
   <!-- Base footprint is on the ground under the robot -->
   <link name="base_footprint"/>

File: vehicle_autonomy/propbot_description/urdf/wheel.urdf.xacro (robot description, xacro)
@@ -53,4 +53,5 @@
 			<kd value="1.0" />
 			<fdir1 value="1 0 0"/>
+      		<material>Gazebo/Black</material>
 		</gazebo>
 		<joint name="${wheel_prefix}_wheel" type="continuous">

Commit message: Adds correct frames for urdf model

File: vehicle_autonomy/propbot_description/urdf/decorations.urdf.xacro (robot description, xacro)
@@ -26,5 +26,5 @@
     <link name="chassis_link">
       <visual>
-        <origin xyz="0 ${base_x_size/2} ${2*wheel_vertical_offset - base_z_size}" rpy="${M_PI/2} 0 0" />
+        <origin xyz="${base_x_size/2} 0 ${2*wheel_vertical_offset - base_z_size}" rpy="${M_PI/2} 0 ${-M_PI/2}" />
         <geometry>
           <mesh filename="package://propbot_description/meshes/propbot_chassis.STL" />
@@ -45,5 +45,5 @@
       <link name="top_plate_link">
         <visual>
-          <origin xyz="0 0 ${top_plate_height}" rpy="0 0 0" />
+          <origin xyz="0 0 ${top_plate_height}" rpy="0 0 ${-M_PI/2}" />
           <geometry>
             <box size="0.001 0.001 0.001"/>

File: vehicle_autonomy/propbot_description/urdf/passive_wheel.urdf.xacro (robot description, xacro)
@@ -26,7 +26,8 @@
 			<!-- Following values extracted from URDF exported from Solidworks -->
 			<inertial>
-				<mass value="2.96542" />
+				<mass value="${wheel_mass*msf}" />
 				<origin xyz="0 0 0" />
-				<inertia  ixx="0.01875" ixy="1.054410E-15" ixz="6.83081E-07" iyy="0.01012" iyz="-4.64239E-08" izz="0.01012" />
+				<inertia  ixx="${0.01875*msf}" ixy="${1.054410E-15*msf}" ixz="${6.83081E-07*msf}"
+				          iyy="${0.01012*msf}" iyz="${-4.64239E-08*msf}" izz="${0.01012*msf}" />
 			</inertial>
 			<visual>
@@ -47,25 +48,18 @@
 		</link>
 		<gazebo reference="${wheel_prefix}_wheel_link">
-			<mu1 value="1.0"/>
-			<mu2 value="1.0"/>
+			<mu1 value="100.0"/>
+			<mu2 value="100.0"/>
 			<kp value="10000000.0" />
 			<kd value="1.0" />
 			<fdir1 value="1 0 0"/>
+      		<material>Gazebo/Black</material>
 		</gazebo>
-		<joint name="${wheel_prefix}_wheel" type="continuous">
+		<joint name="${wheel_prefix}_wheel" type="fixed">
 			<parent link="base_link"/>
 			<child link="${wheel_prefix}_wheel_link"/>
 			<xacro:insert_block name="joint_pose"/>
-			<axis xyz="1 0 0" rpy="0 0 0" />
+			<axis xyz="-1 0 0" rpy="0 0 0" />
+			<dynamics damping="0.0" friction="0.0"/>
 		</joint>
-		<transmission name="${wheel_prefix}_wheel_trans" type="SimpleTransmission">
-			<type>transmission_interface/SimpleTransmission</type>
-			<actuator name="${wheel_prefix}_wheel_motor">
-				<mechanicalReduction>1</mechanicalReduction>
-			</actuator>
-			<joint name="${wheel_prefix}_wheel">
-				<hardwareInterface>hardware_interface/VelocityJointInterface</hardwareInterface>
-			</joint>
-		</transmission>
 	</xacro:macro>
 </robot>

File: vehicle_autonomy/propbot_description/urdf/propbot.urdf.xacro (robot description, xacro)
@@ -28,5 +28,5 @@
 <robot name="propbot" xmlns:xacro="http://ros.org/wiki/xacro">
   <xacro:arg name="laser_enabled" default="false" />
-  <xacro:arg name="laser_xyz" default="$(optenv PROPBOT_VLP-16_XYZ 0.2206 0.0 0)" />
+  <xacro:arg name="laser_xyz" default="$(optenv PROPBOT_VLP-16_XYZ 0.2206 0.0 1.2)" />
   <xacro:arg name="laser_rpy" default="$(optenv PROPBOT_VLP-16_RPY 0.0 0.0 0.0)" />
   <xacro:arg name="rgbd_camera_enabled" default="false" />
@@ -49,5 +49,6 @@
   <xacro:property name="wheel_mass" value="2.96542"/>     <!-- Wheel mass as reported by SW -->
   <xacro:property name="chassis_mass" value="19.52246"/>  <!-- Chassis mass as reported by SW -->
-  <xacro:property name="msf" value="${robot_mass/(chassis_mass + 6*wheel_mass)}"/> <!-- Mass scale factor: use to scale masses and inertial values -->
+  <xacro:property name="msf" value="${robot_mass/(chassis_mass + 6*wheel_mass)}"/>  <!-- Mass scale factor: use to scale masses and inertial values -->
+  <!-- <xacro:property name="msf" value="1"/> Mass scale factor: use to scale masses and inertial values -->
   <!-- Wheel Properties -->
   <xacro:property name="wheel_length" value="0.08975" />
@@ -68,5 +69,5 @@
   <link name="base_link">
     <visual>
-      <origin xyz="0 0 ${base_z_size}" rpy="0 0 0" />
+      <origin xyz="0 0 ${base_z_size}" rpy="0 0 ${-M_PI/2}" />
       <geometry>
         <mesh filename="package://propbot_description/meshes/propbot_base_link.STL" />
@@ -74,13 +75,7 @@
     </visual>
     <collision>
-      <origin xyz="0 ${wheel_central_offset + wheel_length/2} ${base_z_size/4}" rpy="0 0 0" />
+      <origin xyz="0 ${wheel_central_offset + wheel_length/2} ${base_z_size/4}" rpy="0 0 ${-M_PI/2}" />
       <geometry>
         <box size="${base_x_size} ${base_y_size} ${base_z_size/2}"/>
-      </geometry>
-    </collision>
-    <collision>
-      <origin xyz="0 ${wheel_central_offset + wheel_length/2} ${base_z_size*3/4-0.01}" rpy="0 0 0" />
-      <geometry>
-        <box size="${base_x_size*4/5} ${base_y_size} ${base_z_size/2-0.02}"/>
       </geometry>
     </collision>
@@ -103,5 +98,5 @@
     <inertial>
       <mass value="${chassis_mass*msf}"/>
-      <origin xyz="-0.004962 0.106799 0.42243" />
+      <origin xyz="-0.004962 0.10679 0.42243" rpy = "${-M_PI/2} ${-M_PI/2} 0" />
       <inertia ixx="${0.42226*msf}" ixy="${0.00028*msf}" ixz="${-0.00012*msf}"
                iyy="${0.46973*msf}" iyz="${0.00017*msf}" izz="${0.16238*msf}" />
@@ -124,21 +119,21 @@
   </gazebo>
   <!-- Propbot wheel macros -->
-  <xacro:propbot_wheel wheel_prefix="front_right">
-    <origin xyz="${track/2} ${wheel_to_wheel} ${wheel_vertical_offset}" rpy="0 ${M_PI} 0" />
-  </xacro:propbot_wheel>
   <xacro:propbot_wheel wheel_prefix="front_left">
-    <origin xyz="${-track/2} ${wheel_to_wheel} ${wheel_vertical_offset}" rpy="0 0 0" />
-  </xacro:propbot_wheel>
-  <xacro:propbot_passive_wheel wheel_prefix="middle_right">
-    <origin xyz="${track/2} 0 ${wheel_vertical_offset}" rpy="0 ${M_PI} 0" />
-  </xacro:propbot_passive_wheel>
-  <xacro:propbot_passive_wheel wheel_prefix="middle_left">
-    <origin xyz="${-track/2} 0 ${wheel_vertical_offset}" rpy="0 0 0" />
-  </xacro:propbot_passive_wheel>
-  <xacro:propbot_wheel wheel_prefix="rear_right">
-    <origin xyz="${track/2} ${-wheel_to_wheel} ${wheel_vertical_offset}" rpy="0 ${M_PI} 0" />
+    <origin xyz="${track/2} ${wheel_to_wheel} ${wheel_vertical_offset}" rpy="0 0 ${-M_PI/2}" />
   </xacro:propbot_wheel>
   <xacro:propbot_wheel wheel_prefix="rear_left">
-    <origin xyz="${-track/2} ${-wheel_to_wheel} ${wheel_vertical_offset}" rpy="0 0 0" />
+    <origin xyz="${-track/2 + wheel_radius} ${wheel_to_wheel} ${wheel_vertical_offset}" rpy="0 0 ${-M_PI/2}" />
+  </xacro:propbot_wheel>
+  <xacro:propbot_passive_wheel wheel_prefix="middle_left">
+    <origin xyz="0 ${wheel_to_wheel} ${wheel_vertical_offset}" rpy="0 0 ${-M_PI/2}" />
+  </xacro:propbot_passive_wheel>
+  <xacro:propbot_passive_wheel wheel_prefix="middle_right">
+    <origin xyz="0 ${-wheel_to_wheel} ${wheel_vertical_offset}" rpy="0 0 ${-M_PI/2}" />
+  </xacro:propbot_passive_wheel>
+  <xacro:propbot_wheel wheel_prefix="front_right">
+    <origin xyz="${track/2} ${-wheel_to_wheel} ${wheel_vertical_offset}" rpy="0 0 ${-M_PI/2}" />
+  </xacro:propbot_wheel>
+  <xacro:propbot_wheel wheel_prefix="rear_right">
+    <origin xyz="${-track/2 + wheel_radius} ${-wheel_to_wheel} ${wheel_vertical_offset}" rpy="0 0 ${-M_PI/2}" />
   </xacro:propbot_wheel>
   <xacro:propbot_decorate />

File: vehicle_autonomy/propbot_description/urdf/wheel.urdf.xacro (robot description, xacro)
@@ -48,6 +48,6 @@
 		</link>
 		<gazebo reference="${wheel_prefix}_wheel_link">
-			<mu1 value="1.0"/>
-			<mu2 value="1.0"/>
+			<mu1 value="100.0"/>
+			<mu2 value="100.0"/>
 			<kp value="10000000.0" />
 			<kd value="1.0" />
@@ -59,5 +59,5 @@
 			<child link="${wheel_prefix}_wheel_link"/>
 			<xacro:insert_block name="joint_pose"/>
-			<axis xyz="1 0 0" rpy="0 0 0" />
+			<axis xyz="-1 0 0" rpy="0 0 0" />
 		</joint>
 		<transmission name="${wheel_prefix}_wheel_trans" type="SimpleTransmission">

Commit message: Updated wheel spacing and test top plate size

File: vehicle_autonomy/propbot_description/urdf/decorations.urdf.xacro (robot description, xacro)
@@ -47,5 +47,5 @@
           <origin xyz="0 0 ${top_plate_height}" rpy="0 0 ${-M_PI/2}" />
           <geometry>
-            <box size="0.001 0.001 0.001"/>
+            <box size="0.1 0.05 0.001"/>
           </geometry>
           <material name="wheel_material">

File: vehicle_autonomy/propbot_description/urdf/propbot.urdf.xacro (robot description, xacro)
@@ -28,5 +28,5 @@
 <robot name="propbot" xmlns:xacro="http://ros.org/wiki/xacro">
   <xacro:arg name="laser_enabled" default="false" />
-  <xacro:arg name="laser_xyz" default="$(optenv PROPBOT_VLP-16_XYZ 0.2206 0.0 1.2)" />
+  <xacro:arg name="laser_xyz" default="$(optenv PROPBOT_VLP-16_XYZ 0.2206 0.0 0.75)" />
   <xacro:arg name="laser_rpy" default="$(optenv PROPBOT_VLP-16_RPY 0.0 0.0 0.0)" />
   <xacro:arg name="rgbd_camera_enabled" default="false" />
@@ -123,17 +123,17 @@
   </xacro:propbot_wheel>
   <xacro:propbot_wheel wheel_prefix="rear_left">
-    <origin xyz="${-track/2 + wheel_radius} ${wheel_to_wheel} ${wheel_vertical_offset}" rpy="0 0 ${-M_PI/2}" />
+    <origin xyz="${-track/2 + wheel_radius/2} ${wheel_to_wheel} ${wheel_vertical_offset}" rpy="0 0 ${-M_PI/2}" />
   </xacro:propbot_wheel>
   <xacro:propbot_passive_wheel wheel_prefix="middle_left">
-    <origin xyz="0 ${wheel_to_wheel} ${wheel_vertical_offset}" rpy="0 0 ${-M_PI/2}" />
-  </xacro:propbot_passive_wheel>
-  <xacro:propbot_passive_wheel wheel_prefix="middle_right">
-    <origin xyz="0 ${-wheel_to_wheel} ${wheel_vertical_offset}" rpy="0 0 ${-M_PI/2}" />
+    <origin xyz="0 ${wheel_to_wheel + wheel_radius/2} ${wheel_vertical_offset}" rpy="0 0 ${-M_PI/2}" />
   </xacro:propbot_passive_wheel>
   <xacro:propbot_wheel wheel_prefix="front_right">
     <origin xyz="${track/2} ${-wheel_to_wheel} ${wheel_vertical_offset}" rpy="0 0 ${-M_PI/2}" />
   </xacro:propbot_wheel>
+  <xacro:propbot_passive_wheel wheel_prefix="middle_right">
+    <origin xyz="0 ${-wheel_to_wheel + wheel_radius/2} ${wheel_vertical_offset}" rpy="0 0 ${-M_PI/2}" />
+  </xacro:propbot_passive_wheel>
   <xacro:propbot_wheel wheel_prefix="rear_right">
-    <origin xyz="${-track/2 + wheel_radius} ${-wheel_to_wheel} ${wheel_vertical_offset}" rpy="0 0 ${-M_PI/2}" />
+    <origin xyz="${-track/2 + wheel_radius/2} ${-wheel_to_wheel} ${wheel_vertical_offset}" rpy="0 0 ${-M_PI/2}" />
   </xacro:propbot_wheel>
   <xacro:propbot_decorate />

Commit message: Top plate translation

File: vehicle_autonomy/propbot_description/urdf/decorations.urdf.xacro (robot description, xacro)
@@ -45,7 +45,7 @@
       <link name="top_plate_link">
         <visual>
-          <origin xyz="0 0 ${top_plate_height}" rpy="0 0 ${-M_PI/2}" />
+          <origin xyz="${base_x_size/2} ${base_y_size/2} ${top_plate_height}" rpy="0 0 ${-M_PI/2}" />
           <geometry>
-            <box size="0.1 0.05 0.001"/>
+            <box size="0.2 0.1 0.005"/>
           </geometry>
           <material name="wheel_material">
