Commit message: WIP addition of base link weights and inertia

File: vehicle_autonomy/propbot_description/urdf/decorations.urdf.xacro (robot description, xacro)
@@ -45,5 +45,5 @@
       <link name="top_plate_link">
         <visual>
-          <origin xyz="${base_x_size/2} ${base_y_size/2} ${top_plate_height}" rpy="0 0 ${-M_PI/2}" />
+          <origin xyz="${base_x_size/2} 0 ${top_plate_height}" rpy="0 0 0" />
           <geometry>
             <box size="0.2 0.1 0.005"/>

File: vehicle_autonomy/propbot_description/urdf/propbot.urdf.xacro (robot description, xacro)
@@ -22,9 +22,27 @@
 -->
 <!-- NOTES
-==============================================================================================================
 * All values are in metric (m, kg)
 * Specific robot structure values extracted from URDF exported from Solidworks
 -->
 <robot name="propbot" xmlns:xacro="http://ros.org/wiki/xacro">
+  <!--
+  ***********************************************************************************************
+  Default Spawn Settings
+  ***********************************************************************************************
+  -->
+  <xacro:arg name="robot_namespace" default="/" />
+  <xacro:arg name="spawn_lat" default="49.9" />
+  <xacro:arg name="spawn_long" default="8.9" />
+  <!--
+  ***********************************************************************************************
+  Misc. Constants
+  ***********************************************************************************************
+  -->
+  <xacro:property name="M_PI" value="3.14159"/>
+  <!--
+  ***********************************************************************************************
+  Laser and Camera Args
+  ***********************************************************************************************
+  -->
   <xacro:arg name="laser_enabled" default="false" />
   <xacro:arg name="laser_xyz" default="$(optenv PROPBOT_VLP-16_XYZ 0.2206 0.0 0.75)" />
@@ -33,8 +51,9 @@
   <xacro:arg name="rgbd_camera_xyz" default="$(optenv PROPBOT_REALSENSE_XYZ 0 0 0)" />
   <xacro:arg name="rgbd_camera_rpy" default="$(optenv PROPBOT_REALSENSE_RPY 0 0.18 3.14)" />
-  <xacro:arg name="robot_namespace" default="/" />
-  <xacro:arg name="spawn_lat" default="49.9" />
-  <xacro:arg name="spawn_long" default="8.9" />
-  <!-- Included URDF/XACRO Files -->
+  <!--
+  ***********************************************************************************************
+  Included URDF/XACRO Files
+  ***********************************************************************************************
+  -->
   <xacro:include filename="$(find propbot_description)/urdf/decorations.urdf.xacro" />
   <xacro:include filename="$(find propbot_description)/urdf/wheel.urdf.xacro" />
@@ -43,16 +62,39 @@
   <xacro:include filename="$(find propbot_description)/urdf/accessories/sensor_arch.urdf.xacro"/>
   <xacro:include filename="$(find propbot_description)/urdf/accessories/VLP-16_mount.urdf.xacro"/>
-  <!-- Define Constant(s) -->
-  <xacro:property name="M_PI" value="3.14159"/>
-  <!-- Inertia and Mass Scaling -->
-  <xacro:property name="robot_mass" value="82"/>          <!-- Approximate robot mass is approx 82kg, SolidWorks model incorrect -->
-  <xacro:property name="wheel_mass" value="2.96542"/>     <!-- Wheel mass as reported by SW -->
-  <!-- <xacro:property name="chassis_mass" value="19.52246"/>   -->
-  <!-- Chassis mass as reported by SW -->
-  <xacro:property name="chassis_mass" value="70.00"/>
-  <!-- <xacro:property name="msf" value="${robot_mass/(chassis_mass + 6*wheel_mass)}"/>   -->
-  <!-- Mass scale factor: use to scale masses and inertial values -->
-  <xacro:property name="msf" value="1"/>
-  <!-- Mass scale factor: use to scale masses and inertial values -->
+  <!--
+  ***********************************************************************************************
+  Mass and Inertial Values and Scaling
+  ***********************************************************************************************
+  Values as reported by SolidWorks
+  -->
+  <!-- Approximate REAL robot mass -->
+  <xacro:property name="robot_mass" value="70.0"/>
+  <!-- SW reported mass values -->
+  <xacro:property name="base_link_mass" value="0.96268" />
+  <xacro:property name="chassis_mass" value="19.52246"/>
+  <xacro:property name="wheel_mass" value="2.96542"/>
+  <!-- Base link inertia-->
+  <xacro:property name="base_ixx" value="0.083320" />
+  <xacro:property name="base_ixy" value="-1.882647E-14" />
+  <xacro:property name="base_ixz" value="2.527076E-19" />
+  <xacro:property name="base_iyy" value="0.003905" />
+  <xacro:property name="base_iyz" value="7.039418E-19" />
+  <xacro:property name="base_izz" value="0.087218" />
+   <!-- Chassis link inertia-->
+  <xacro:property name="chassis_ixx" value="0.42226" />
+  <xacro:property name="chassis_ixy" value="0.00028" />
+  <xacro:property name="chassis_ixz" value="-0.00012" />
+  <xacro:property name="chassis_iyy" value="0.46973" />
+  <xacro:property name="chassis_iyz" value="0.00017" />
+  <xacro:property name="chassis_izz" value="0.16238" />
+  <!-- Robot frame mass scale factor: use to scale chassis and base link masses and inertial values -->
+  <xacro:property name="frame_msf" value="${robot_mass/chassis_mass}" />
+  <!-- Wheel mass scale factor: use to scale wheel masses and inertial values -->
+  <xacro:property name="wheel_msf" value="1" />
+  <!--
+  ***********************************************************************************************
+  Wheel Properties and Mounting Specifications
+  ***********************************************************************************************
+  -->
   <!-- Wheel Properties -->
   <xacro:property name="wheel_length" value="0.08975" />
@@ -63,11 +105,30 @@
   <xacro:property name="wheel_vertical_offset" value="${wheel_radius}" /> <!-- axle to ground distance -->
   <xacro:property name="wheel_central_offset" value="0.0533" /> <!-- offset from the center -->
-  <!-- Base Size -->
+  <!--
+  ***********************************************************************************************
+  Base Size Specifications
+  ***********************************************************************************************
+  The "shadow" of the robot
+  -->
   <xacro:property name="base_x_size" value="0.9820" /> <!-- x is front to back -->
   <xacro:property name="base_y_size" value="0.8278" /> <!-- y is side to side -->
   <xacro:property name="base_z_size" value="0.1369" /> <!-- height of the bottom battery plate from the ground -->
-  <!-- Sensor Mounting Values -->
+  <!--
+  ***********************************************************************************************
+  Sensor Mounting Specifications
+  ***********************************************************************************************
+  -->
   <xacro:property name="top_plate_height" value="${0.24845 + wheel_radius}" /> <!-- height from the ground to the top plate -->
   <xacro:property name="top_plate_front" value="${base_x_size/2}" /> <!-- distance from the origin to the front of the robot -->
+  <!--
+  ***********************************************************************************************
+  Linking and Joint Specification
+  ***********************************************************************************************
+  The various links and joints are created and put together
+  -->
+  <!--
+  Base Link
+  ======================================================================
+  -->
   <!-- Base link is the center of the robot's bottom plate -->
   <link name="base_link">
@@ -96,13 +157,21 @@
     <child link="base_footprint" />
   </joint>
-  <!-- Interial link stores the robot's inertial information
-       For this case, the mass, origin, and inertia values of the main chassis is used
+  <!--
+  Inertial Link
+  ======================================================================
+  Interial link stores the robot's inertial information
+  For this case, the mass, origin, and inertia values of the main chassis is used
   -->
   <link name="inertial_link">
     <inertial>
-      <mass value="${chassis_mass*msf}"/>
+      <mass value="${(chassis_mass + base_link_mass) * frame_msf}"/>
       <origin xyz="-0.004962 0.10679 0.42243" rpy = "${-M_PI/2} ${-M_PI/2} 0" />
-      <inertia ixx="${0.42226*msf}" ixy="${0.00028*msf}" ixz="${-0.00012*msf}"
-               iyy="${0.46973*msf}" iyz="${0.00017*msf}" izz="${0.16238*msf}" />
+      <inertia
+        ixx="${(base_ixx + chassis_ixx) * frame_msf}"
+        ixy="${(base_ixy + chassis_ixy) * frame_msf}"
+        ixz="${(base_ixz + chassis_ixz) * frame_msf}"
+        iyy="${(base_iyy + chassis_iyy) * frame_msf}"
+        iyz="${(base_iyz + chassis_iyz) * frame_msf}"
+        izz="${(base_izz + chassis_izz) * frame_msf}" />
     </inertial>
   </link>
@@ -112,6 +181,10 @@
     <child link="inertial_link" />
   </joint>
-  <!-- IMU Link is the standard mounting position for the UM6 IMU.-->
-  <!-- Can be modified with environment variables in /etc/ros/setup.bash -->
+  <!--
+  IMU Link
+  ======================================================================
+  IMU Link is the standard mounting position for the UM6 IMU.
+  Can be modified with environment variables in /etc/ros/setup.bash
+  -->
   <link name="imu_link"/>
   <joint name="imu_joint" type="fixed">
@@ -122,5 +195,16 @@
   <gazebo reference="imu_link">
   </gazebo>
-  <!-- Propbot wheel macros -->
+  <!--
+  Wheels
+  ======================================================================
+  -->
+  <!-- Right -->
+  <xacro:propbot_wheel wheel_prefix="front_right">
+    <origin xyz="${track/2} ${-wheel_to_wheel} ${wheel_vertical_offset}" rpy="0 0 ${-M_PI/2}" />
+  </xacro:propbot_wheel>
+  <xacro:propbot_wheel wheel_prefix="rear_right">
+    <origin xyz="${-track/2 + (2/3)*wheel_radius} ${-wheel_to_wheel} ${wheel_vertical_offset}" rpy="0 0 ${-M_PI/2}" />
+  </xacro:propbot_wheel>
+  <!-- Left -->
   <xacro:propbot_wheel wheel_prefix="front_left">
     <origin xyz="${track/2} ${wheel_to_wheel} ${wheel_vertical_offset}" rpy="0 0 ${-M_PI/2}" />
@@ -129,4 +213,5 @@
     <origin xyz="${-track/2 + (2/3)*wheel_radius} ${wheel_to_wheel} ${wheel_vertical_offset}" rpy="0 0 ${-M_PI/2}" />
   </xacro:propbot_wheel>
+  <!-- Middle (passives) -->
   <xacro:propbot_passive_wheel wheel_prefix="left">
     <origin xyz="${wheel_radius/3} ${wheel_to_wheel} ${wheel_vertical_offset}" rpy="0 0 ${-M_PI/2}" />
@@ -135,11 +220,10 @@
     <origin xyz="${wheel_radius/3} ${-wheel_to_wheel} ${wheel_vertical_offset}" rpy="0 0 ${-M_PI/2}" />
   </xacro:propbot_passive_wheel>
-  <xacro:propbot_wheel wheel_prefix="front_right">
-    <origin xyz="${track/2} ${-wheel_to_wheel} ${wheel_vertical_offset}" rpy="0 0 ${-M_PI/2}" />
-  </xacro:propbot_wheel>
-  <xacro:propbot_wheel wheel_prefix="rear_right">
-    <origin xyz="${-track/2 + (2/3)*wheel_radius} ${-wheel_to_wheel} ${wheel_vertical_offset}" rpy="0 0 ${-M_PI/2}" />
-  </xacro:propbot_wheel>
+  <!-- Decorate the robot -->
   <xacro:propbot_decorate />
+  <!--
+  Laser and Camera
+  ======================================================================
+  -->
   <xacro:if value="$(arg laser_enabled)">
     <VLP-16_mount prefix="base" />
@@ -158,4 +242,10 @@
      </realsense_d435>
   </xacro:if>
+  <!--
+  ***********************************************************************************************
+  Gazebo Specifications
+  ***********************************************************************************************
+  -->
+  <!-- Motion controller -->
   <gazebo>
     <plugin name="gazebo_ros_control" filename="libgazebo_ros_control.so">
@@ -163,4 +253,5 @@
     </plugin>
   </gazebo>
+  <!-- IMU controller -->
   <gazebo>
     <plugin name="imu_controller" filename="libhector_gazebo_ros_imu.so">
@@ -177,4 +268,5 @@
     </plugin>
   </gazebo>
+  <!-- GPS controller -->
   <gazebo>
     <plugin name="gps_controller" filename="libhector_gazebo_ros_gps.so">

File: vehicle_autonomy/propbot_description/urdf/wheel.urdf.xacro (robot description, xacro)
@@ -26,8 +26,8 @@
 			<!-- Following values extracted from URDF exported from Solidworks -->
 			<inertial>
-				<mass value="${wheel_mass*msf}" />
+				<mass value="${wheel_mass*wheel_msf}" />
 				<origin xyz="0 0 0" />
-				<inertia  ixx="${0.01875*msf}" ixy="${1.054410E-15*msf}" ixz="${6.83081E-07*msf}"
-				          iyy="${0.01012*msf}" iyz="${-4.64239E-08*msf}" izz="${0.01012*msf}" />
+				<inertia  ixx="${0.01875*wheel_msf}" ixy="${1.054410E-15*wheel_msf}" ixz="${6.83081E-07*wheel_msf}"
+				          iyy="${0.01012*wheel_msf}" iyz="${-4.64239E-08*wheel_msf}" izz="${0.01012*wheel_msf}" />
 			</inertial>
 			<visual>

Commit message: Fixed top plate location

File: vehicle_autonomy/propbot_description/urdf/decorations.urdf.xacro (robot description, xacro)
@@ -22,5 +22,16 @@
 -->
 <robot name="propbot_decorations" xmlns:xacro="http://ros.org/wiki/xacro">
+  <!--
+  ***********************************************************************************************
+  Propbot Decoration
+  ***********************************************************************************************
+  The chassis and sensors are considered "decorations" on the base_link. A macro is defined below
+  to execute this decoration in one step in `propbot.urdf.xacro`
+  -->
   <xacro:macro name="propbot_decorate">
+    <!--
+    Chassis
+    ======================================================================
+    -->
     <!-- Spawn Propbot chassis -->
     <link name="chassis_link">
@@ -41,11 +52,16 @@
       <child link="chassis_link" />
     </joint>
+    <!--
+    Top plate
+    ======================================================================
+    A tiny plate use to link the sensors to the robot
+    -->
     <xacro:if value="$(optenv PROPBOT_TOP_PLATE_ENABLED true)">
-      <!-- Spawn "invisible" the top plate -->
+      <!-- Spawn the top plate -->
       <link name="top_plate_link">
         <visual>
-          <origin xyz="${base_x_size/2} 0 ${top_plate_height}" rpy="0 0 0" />
+          <origin xyz="${base_x_size/2} ${-base_y_size/2 + 0.027} ${top_plate_height}" rpy="0 0 0" />
           <geometry>
-            <box size="0.2 0.1 0.005"/>
+            <box size="0.01 0.01 0.001"/>
           </geometry>
           <material name="wheel_material">

File: vehicle_autonomy/propbot_description/urdf/passive_wheel.urdf.xacro (robot description, xacro)
@@ -26,7 +26,13 @@
 			<!-- Following values extracted from URDF exported from Solidworks -->
 			<inertial>
-				<mass value="${wheel_mass*msf}" />
+				<mass value="${wheel_mass * wheel_msf}" />
 				<origin xyz="0 0 0" />
-				<inertia ixx="${0.01875*msf}" ixy="${1.054410E-15*msf}" ixz="${6.83081E-07*msf}" iyy="${0.01012*msf}" iyz="${-4.64239E-08*msf}" izz="${0.01012*msf}" />
+				<inertia
+					ixx="${0.01875 * wheel_msf}"
+					ixy="${1.054410E-15 * wheel_msf}"
+					ixz="${6.83081E-07 * wheel_msf}"
+					iyy="${0.01012 * wheel_msf}"
+					iyz="${-4.64239E-08 * wheel_msf}"
+					izz="${0.01012 * wheel_msf}" />
 			</inertial>
 			<visual>

File: vehicle_autonomy/propbot_description/urdf/wheel.urdf.xacro (robot description, xacro)
@@ -26,8 +26,8 @@
 			<!-- Following values extracted from URDF exported from Solidworks -->
 			<inertial>
-				<mass value="${wheel_mass*wheel_msf}" />
+				<mass value="${wheel_mass * wheel_msf}" />
 				<origin xyz="0 0 0" />
-				<inertia  ixx="${0.01875*wheel_msf}" ixy="${1.054410E-15*wheel_msf}" ixz="${6.83081E-07*wheel_msf}"
-				          iyy="${0.01012*wheel_msf}" iyz="${-4.64239E-08*wheel_msf}" izz="${0.01012*wheel_msf}" />
+				<inertia  ixx="${0.01875 * wheel_msf}" ixy="${1.054410E-15 * wheel_msf}" ixz="${6.83081E-07 * wheel_msf}"
+				          iyy="${0.01012 * wheel_msf}" iyz="${-4.64239E-08 * wheel_msf}" izz="${0.01012 * wheel_msf}" />
 			</inertial>
 			<visual>
