Commit message: Fixes wheel issue, adds passive wheel file

File: vehicle_autonomy/propbot_description/urdf/passive_wheel.urdf.xacro (robot description, xacro)
@@ -21,6 +21,6 @@
 ARISING IN ANY WAY OUT OF THE USE OF THIS SOFTWARE, EVEN IF ADVISED OF THE POSSIBILITY OF SUCH DAMAGE.
 -->
-<robot xmlns:xacro="http://ros.org/wiki/xacro" name="propbot_wheel">
-	<xacro:macro name="propbot_wheel" params="wheel_prefix *joint_pose">
+<robot xmlns:xacro="http://ros.org/wiki/xacro" name="propbot_passive_wheel">
+	<xacro:macro name="propbot_passive_wheel" params="wheel_prefix *joint_pose">
 		<link name="${wheel_prefix}_wheel_link">
 			<!-- Following values extracted from URDF exported from Solidworks -->

File: vehicle_autonomy/propbot_description/urdf/propbot.urdf.xacro (robot description, xacro)
@@ -28,5 +28,5 @@
 <robot name="propbot" xmlns:xacro="http://ros.org/wiki/xacro">
   <xacro:arg name="laser_enabled" default="false" />
-  <xacro:arg name="laser_xyz" default="$(optenv PROPBOT_VLP-16_XYZ 0.2206 0.0 0.00635)" />
+  <xacro:arg name="laser_xyz" default="$(optenv PROPBOT_VLP-16_XYZ 0.2206 0.0 1.4)" />
   <xacro:arg name="laser_rpy" default="$(optenv PROPBOT_VLP-16_RPY 0.0 0.0 0.0)" />
   <xacro:arg name="rgbd_camera_enabled" default="false" />
@@ -39,4 +39,5 @@
   <xacro:include filename="$(find propbot_description)/urdf/decorations.urdf.xacro" />
   <xacro:include filename="$(find propbot_description)/urdf/wheel.urdf.xacro" />
+  <xacro:include filename="$(find propbot_description)/urdf/passive_wheel.urdf.xacro" />
   <xacro:include filename="$(find propbot_description)/urdf/accessories/realsense_d435.urdf.xacro"/>
   <xacro:include filename="$(find propbot_description)/urdf/accessories/sensor_arch.urdf.xacro"/>
@@ -45,4 +46,5 @@
   <xacro:property name="M_PI" value="3.14159"/>
   <!-- Wheel Properties -->
+  <xacro:property name="wheel_length" value="0.08975" />
   <xacro:property name="wheel_radius" value="0.127" />
   <!-- Wheel Mounting Positions -->
@@ -118,10 +120,10 @@
     <origin xyz="${-track/2} ${wheel_to_wheel + wheel_central_offset} ${wheel_vertical_offset}" rpy="0 0 0" />
   </xacro:propbot_wheel>
-  <xacro:propbot_wheel wheel_prefix="middle_left">
+  <xacro:propbot_passive_wheel wheel_prefix="middle_left">
     <origin xyz="${track/2} ${wheel_central_offset} ${wheel_vertical_offset}" rpy="0 ${M_PI} 0" />
-  </xacro:propbot_wheel>
-  <xacro:propbot_wheel wheel_prefix="middle_right">
+  </xacro:propbot_passive_wheel>
+  <xacro:propbot_passive_wheel wheel_prefix="middle_right">
     <origin xyz="${-track/2} ${wheel_central_offset} ${wheel_vertical_offset}" rpy="0 0 0" />
-  </xacro:propbot_wheel>
+  </xacro:propbot_passive_wheel>
   <xacro:propbot_wheel wheel_prefix="rear_left">
     <origin xyz="${track/2} ${-wheel_to_wheel + wheel_central_offset} ${wheel_vertical_offset}" rpy="0 ${M_PI} 0" />

Commit message: Adds passive wheels that mimic rear wheels

File: vehicle_autonomy/propbot_description/urdf/passive_wheel.urdf.xacro (robot description, xacro)
@@ -1,3 +1,3 @@
-<?xml version="1.0"?>
+<?xml version="1.0" ?>
 <!--
 Software License Agreement (BSD)
@@ -28,15 +28,15 @@
 				<mass value="${wheel_mass*msf}" />
 				<origin xyz="0 0 0" />
-				<inertia  ixx="${0.01875*msf}" ixy="${1.054410E-15*msf}" ixz="${6.83081E-07*msf}"
-				          iyy="${0.01012*msf}" iyz="${-4.64239E-08*msf}" izz="${0.01012*msf}" />
+				<inertia ixx="${0.01875*msf}" ixy="${1.054410E-15*msf}" ixz="${6.83081E-07*msf}" iyy="${0.01012*msf}" iyz="${-4.64239E-08*msf}" izz="${0.01012*msf}" />
 			</inertial>
 			<visual>
 				<origin xyz="0 0 0" rpy="0 0 0" />
 				<geometry>
-					<mesh filename="package://propbot_description/meshes/propbot_wheel.STL" />>
+					<mesh filename="package://propbot_description/meshes/propbot_wheel.STL" />
+					>
 				</geometry>
 				<material name="wheel_material">
-				  <color rgba="0.109804 0.109804 0.109804 1" />
-      			</material>
+					<color rgba="0.109804 0.109804 0.109804 1" />
+				</material>
 			</visual>
 			<collision>
@@ -48,17 +48,17 @@
 		</link>
 		<gazebo reference="${wheel_prefix}_wheel_link">
-			<mu1 value="100.0"/>
-			<mu2 value="100.0"/>
+			<mu1 value="100.0" />
+			<mu2 value="100.0" />
 			<kp value="10000000.0" />
 			<kd value="1.0" />
-			<fdir1 value="1 0 0"/>
-      		<material>Gazebo/Black</material>
+			<fdir1 value="1 0 0" />
+			<material>Gazebo/Black</material>
 		</gazebo>
-		<joint name="${wheel_prefix}_wheel" type="fixed">
-			<parent link="base_link"/>
-			<child link="${wheel_prefix}_wheel_link"/>
-			<xacro:insert_block name="joint_pose"/>
+		<joint name="${wheel_prefix}_wheel" type="continuous">
+			<parent link="base_link" />
+			<child link="${wheel_prefix}_wheel_link" />
+			<xacro:insert_block name="joint_pose" />
+			<mimic joint="rear_${wheel_prefix}_wheel"></mimic>
 			<axis xyz="-1 0 0" rpy="0 0 0" />
-			<dynamics damping="0.0" friction="0.0"/>
 		</joint>
 	</xacro:macro>

File: vehicle_autonomy/propbot_description/urdf/propbot.urdf.xacro (robot description, xacro)
@@ -125,13 +125,13 @@
     <origin xyz="${-track/2 + wheel_radius/2} ${wheel_to_wheel} ${wheel_vertical_offset}" rpy="0 0 ${-M_PI/2}" />
   </xacro:propbot_wheel>
-  <xacro:propbot_passive_wheel wheel_prefix="middle_left">
-    <origin xyz="0 ${wheel_to_wheel + wheel_radius/2} ${wheel_vertical_offset}" rpy="0 0 ${-M_PI/2}" />
+  <xacro:propbot_passive_wheel wheel_prefix="left">
+    <origin xyz="0 ${wheel_to_wheel} ${wheel_vertical_offset}" rpy="0 0 ${-M_PI/2}" />
+  </xacro:propbot_passive_wheel>
+  <xacro:propbot_passive_wheel wheel_prefix="right">
+    <origin xyz="0 ${-wheel_to_wheel} ${wheel_vertical_offset}" rpy="0 0 ${-M_PI/2}" />
   </xacro:propbot_passive_wheel>
   <xacro:propbot_wheel wheel_prefix="front_right">
     <origin xyz="${track/2} ${-wheel_to_wheel} ${wheel_vertical_offset}" rpy="0 0 ${-M_PI/2}" />
   </xacro:propbot_wheel>
-  <xacro:propbot_passive_wheel wheel_prefix="middle_right">
-    <origin xyz="0 ${-wheel_to_wheel + wheel_radius/2} ${wheel_vertical_offset}" rpy="0 0 ${-M_PI/2}" />
-  </xacro:propbot_passive_wheel>
   <xacro:propbot_wheel wheel_prefix="rear_right">
     <origin xyz="${-track/2 + wheel_radius/2} ${-wheel_to_wheel} ${wheel_vertical_offset}" rpy="0 0 ${-M_PI/2}" />

Commit message: mu1=100; changed inertial link's origin

File: vehicle_autonomy/propbot_description/urdf/passive_wheel.urdf.xacro (robot description, xacro)
@@ -54,5 +54,5 @@
 		</link>
 		<gazebo reference="${wheel_prefix}_wheel_link">
-			<mu1 value="75.0" />
+			<mu1 value="100.0" />
 			<mu2 value="100.0" />
 			<kp value="10000000.0" />

File: vehicle_autonomy/propbot_description/urdf/propbot.urdf.xacro (robot description, xacro)
@@ -166,5 +166,5 @@
     <inertial>
       <mass value="${(chassis_mass + base_link_mass) * frame_msf}"/>
-      <origin xyz="-0.004962 0.10679 0.42243" rpy = "${-M_PI/2} ${-M_PI/2} 0" />
+      <origin xyz="0 0 0.42243" rpy = "${-M_PI/2} ${-M_PI/2} 0" />
       <inertia
         ixx="${(base_ixx + chassis_ixx) * frame_msf}"

File: vehicle_autonomy/propbot_description/urdf/wheel.urdf.xacro (robot description, xacro)
@@ -48,5 +48,5 @@
 		</link>
 		<gazebo reference="${wheel_prefix}_wheel_link">
-			<mu1 value="75.0"/>
+			<mu1 value="100.0"/>
 			<mu2 value="100.0"/>
 			<kp value="10000000.0" />

Commit message: Simplified some hweel inertia components to 0

File: vehicle_autonomy/propbot_description/urdf/passive_wheel.urdf.xacro (robot description, xacro)
@@ -30,8 +30,8 @@
 				<inertia
 					ixx="${0.01875 * wheel_msf}"
-					ixy="${1.054410E-15 * wheel_msf}"
-					ixz="${6.83081E-07 * wheel_msf}"
+					ixy="${0 * wheel_msf}"
+					ixz="${0 * wheel_msf}"
 					iyy="${0.01012 * wheel_msf}"
-					iyz="${-4.64239E-08 * wheel_msf}"
+					iyz="${0 * wheel_msf}"
 					izz="${0.01012 * wheel_msf}" />
 			</inertial>
@@ -40,5 +40,4 @@
 				<geometry>
 					<mesh filename="package://propbot_description/meshes/propbot_wheel.STL" />
-					>
 				</geometry>
 				<material name="wheel_material">
@@ -47,5 +46,5 @@
 			</visual>
 			<collision>
-				<origin xyz="0 0 0" rpy="${M_PI/2} 0 0" />
+				<origin xyz="0 0 0" rpy="0 0 0" />
 				<geometry>
 					<cylinder length="${wheel_length}" radius="${wheel_radius}" />

File: vehicle_autonomy/propbot_description/urdf/wheel.urdf.xacro (robot description, xacro)
@@ -28,11 +28,16 @@
 				<mass value="${wheel_mass * wheel_msf}" />
 				<origin xyz="0 0 0" />
-				<inertia  ixx="${0.01875 * wheel_msf}" ixy="${1.054410E-15 * wheel_msf}" ixz="${6.83081E-07 * wheel_msf}"
-				          iyy="${0.01012 * wheel_msf}" iyz="${-4.64239E-08 * wheel_msf}" izz="${0.01012 * wheel_msf}" />
+				<inertia
+					ixx="${0.01875 * wheel_msf}"
+					ixy="${0 * wheel_msf}"
+					ixz="${0 * wheel_msf}"
+					iyy="${0.01012 * wheel_msf}"
+					iyz="${0 * wheel_msf}"
+					izz="${0.01012 * wheel_msf}" />
 			</inertial>
 			<visual>
 				<origin xyz="0 0 0" rpy="0 0 0" />
 				<geometry>
-					<mesh filename="package://propbot_description/meshes/propbot_wheel.STL" />>
+					<mesh filename="package://propbot_description/meshes/propbot_wheel.STL" />
 				</geometry>
 				<material name="wheel_material">
@@ -41,5 +46,5 @@
 			</visual>
 			<collision>
-				<origin xyz="0 0 0" rpy="${M_PI/2} 0 0" />
+				<origin xyz="0 0 0" rpy="0 0 0" />
 				<geometry>
 					<cylinder length="${wheel_length}" radius="${wheel_radius}" />

Commit message: Reduced mu2, removed chassis Ixy component

File: vehicle_autonomy/propbot_description/urdf/passive_wheel.urdf.xacro (robot description, xacro)
@@ -54,5 +54,5 @@
 		<gazebo reference="${wheel_prefix}_wheel_link">
 			<mu1 value="100.0" />
-			<mu2 value="1000.0" />
+			<mu2 value="100.0" />
 			<kp value="10000000.0" />
 			<kd value="1.0" />

File: vehicle_autonomy/propbot_description/urdf/propbot.urdf.xacro (robot description, xacro)
@@ -92,5 +92,5 @@
    <!-- Chassis link inertia-->
   <xacro:property name="chassis_ixx" value="0.42226" />
-  <xacro:property name="chassis_ixy" value="0.00028" />
+  <xacro:property name="chassis_ixy" value="0" />
   <xacro:property name="chassis_ixz" value="0" />
   <xacro:property name="chassis_iyy" value="0.46973" />

File: vehicle_autonomy/propbot_description/urdf/wheel.urdf.xacro (robot description, xacro)
@@ -54,5 +54,5 @@
 		<gazebo reference="${wheel_prefix}_wheel_link">
 			<mu1 value="100.0"/>
-			<mu2 value="1000.0"/>
+			<mu2 value="100.0"/>
 			<kp value="10000000.0" />
 			<kd value="1.0" />

Commit message: Moved inertial origin front and left

File: vehicle_autonomy/propbot_description/urdf/passive_wheel.urdf.xacro (robot description, xacro)
@@ -54,5 +54,5 @@
 		<gazebo reference="${wheel_prefix}_wheel_link">
 			<mu1 value="100.0" />
-			<mu2 value="1000.0" />
+			<mu2 value="350.0" />
 			<kp value="10000000.0" />
 			<kd value="1.0" />

File: vehicle_autonomy/propbot_description/urdf/propbot.urdf.xacro (robot description, xacro)
@@ -166,5 +166,5 @@
     <inertial>
       <mass value="${(chassis_mass + base_link_mass) * frame_msf}"/>
-      <origin xyz="0.027 0 0.42243" rpy = "${-M_PI/2} ${-M_PI/2} 0" />
+      <origin xyz="0.027 0.01 0.42243" rpy = "${-M_PI/2} ${-M_PI/2} 0" />
       <inertia
         ixx="${(base_ixx + chassis_ixx) * frame_msf}"

File: vehicle_autonomy/propbot_description/urdf/wheel.urdf.xacro (robot description, xacro)
@@ -54,5 +54,5 @@
 		<gazebo reference="${wheel_prefix}_wheel_link">
 			<mu1 value="100.0"/>
-			<mu2 value="1000.0"/>
+			<mu2 value="350.0"/>
 			<kp value="10000000.0" />
 			<kd value="1.0" />

Commit message: Urdf balance fixes (#173)
adjusted inertial values for the chassis, base plate, and wheels, and shifted the inertial origin

File: vehicle_autonomy/propbot_description/urdf/passive_wheel.urdf.xacro (robot description, xacro)
@@ -30,9 +30,9 @@
 				<inertia
 					ixx="${0.01875 * wheel_msf}"
-					ixy="${1.054410E-15 * wheel_msf}"
-					ixz="${6.83081E-07 * wheel_msf}"
+					ixy="${0 * wheel_msf}"
+					ixz="${0 * wheel_msf}"
 					iyy="${0.01012 * wheel_msf}"
-					iyz="${-4.64239E-08 * wheel_msf}"
-					izz="${0.01012 * wheel_msf}" />
+					iyz="${0 * wheel_msf}"
+					izz="${0 * wheel_msf}" />
 			</inertial>
 			<visual>
@@ -40,5 +40,4 @@
 				<geometry>
 					<mesh filename="package://propbot_description/meshes/propbot_wheel.STL" />
-					>
 				</geometry>
 				<material name="wheel_material">
@@ -47,5 +46,5 @@
 			</visual>
 			<collision>
-				<origin xyz="0 0 0" rpy="${M_PI/2} 0 0" />
+				<origin xyz="0 0 0" rpy="0 0 0" />
 				<geometry>
 					<cylinder length="${wheel_length}" radius="${wheel_radius}" />

File: vehicle_autonomy/propbot_description/urdf/propbot.urdf.xacro (robot description, xacro)
@@ -85,15 +85,15 @@
   <!-- Base link inertia-->
   <xacro:property name="base_ixx" value="0.083320" />
-  <xacro:property name="base_ixy" value="-1.882647E-14" />
-  <xacro:property name="base_ixz" value="2.527076E-19" />
+  <xacro:property name="base_ixy" value="0" />
+  <xacro:property name="base_ixz" value="0" />
   <xacro:property name="base_iyy" value="0.003905" />
-  <xacro:property name="base_iyz" value="7.039418E-19" />
+  <xacro:property name="base_iyz" value="0" />
   <xacro:property name="base_izz" value="0.087218" />
    <!-- Chassis link inertia-->
   <xacro:property name="chassis_ixx" value="0.42226" />
   <xacro:property name="chassis_ixy" value="0.00028" />
-  <xacro:property name="chassis_ixz" value="-0.00012" />
+  <xacro:property name="chassis_ixz" value="0" />
   <xacro:property name="chassis_iyy" value="0.46973" />
-  <xacro:property name="chassis_iyz" value="0.00017" />
+  <xacro:property name="chassis_iyz" value="0" />
   <xacro:property name="chassis_izz" value="0.16238" />
   <!-- Robot frame mass scale factor: use to scale chassis and base link masses and inertial values -->
@@ -166,5 +166,5 @@
     <inertial>
       <mass value="${(chassis_mass + base_link_mass) * frame_msf}"/>
-      <origin xyz="-0.004962 0.10679 0.42243" rpy = "${-M_PI/2} ${-M_PI/2} 0" />
+      <origin xyz="0.027 -0.01 0.42243" rpy = "${-M_PI/2} ${-M_PI/2} 0" />
       <inertia
         ixx="${(base_ixx + chassis_ixx) * frame_msf}"
@@ -201,22 +201,22 @@
   <!-- Right -->
   <xacro:propbot_wheel wheel_prefix="front_right">
-    <origin xyz="${track/2} ${-wheel_to_wheel} ${wheel_vertical_offset}" rpy="0 0 ${-M_PI/2}" />
+    <origin xyz="${track/2} ${-(wheel_to_wheel + wheel_length/2)} ${wheel_vertical_offset}" rpy="0 0 ${-M_PI/2}" />
   </xacro:propbot_wheel>
   <xacro:propbot_wheel wheel_prefix="rear_right">
-    <origin xyz="${-track/2 + (2/3)*wheel_radius} ${-wheel_to_wheel} ${wheel_vertical_offset}" rpy="0 0 ${-M_PI/2}" />
+    <origin xyz="${-track/2 + (2/3)*wheel_radius} ${-(wheel_to_wheel + wheel_length/2)} ${wheel_vertical_offset}" rpy="0 0 ${-M_PI/2}" />
   </xacro:propbot_wheel>
   <!-- Left -->
   <xacro:propbot_wheel wheel_prefix="front_left">
-    <origin xyz="${track/2} ${wheel_to_wheel} ${wheel_vertical_offset}" rpy="0 0 ${-M_PI/2}" />
+    <origin xyz="${track/2} ${wheel_to_wheel + wheel_length/2} ${wheel_vertical_offset}" rpy="0 0 ${-M_PI/2}" />
   </xacro:propbot_wheel>
   <xacro:propbot_wheel wheel_prefix="rear_left">
-    <origin xyz="${-track/2 + (2/3)*wheel_radius} ${wheel_to_wheel} ${wheel_vertical_offset}" rpy="0 0 ${-M_PI/2}" />
+    <origin xyz="${-track/2 + (2/3)*wheel_radius} ${wheel_to_wheel + wheel_length/2} ${wheel_vertical_offset}" rpy="0 0 ${-M_PI/2}" />
   </xacro:propbot_wheel>
   <!-- Middle (passives) -->
   <xacro:propbot_passive_wheel wheel_prefix="left">
-    <origin xyz="${wheel_radius/3} ${wheel_to_wheel} ${wheel_vertical_offset}" rpy="0 0 ${-M_PI/2}" />
+    <origin xyz="0.027 ${wheel_to_wheel + wheel_length/2} ${wheel_vertical_offset + wheel_radius/10}" rpy="0 0 ${-M_PI/2}" />
   </xacro:propbot_passive_wheel>
   <xacro:propbot_passive_wheel wheel_prefix="right">
-    <origin xyz="${wheel_radius/3} ${-wheel_to_wheel} ${wheel_vertical_offset}" rpy="0 0 ${-M_PI/2}" />
+    <origin xyz="0.027 ${-(wheel_to_wheel + wheel_length/2)} ${wheel_vertical_offset + wheel_radius/10}" rpy="0 0 ${-M_PI/2}" />
   </xacro:propbot_passive_wheel>
   <!-- Decorate the robot -->

File: vehicle_autonomy/propbot_description/urdf/wheel.urdf.xacro (robot description, xacro)
@@ -28,11 +28,16 @@
 				<mass value="${wheel_mass * wheel_msf}" />
 				<origin xyz="0 0 0" />
-				<inertia  ixx="${0.01875 * wheel_msf}" ixy="${1.054410E-15 * wheel_msf}" ixz="${6.83081E-07 * wheel_msf}"
-				          iyy="${0.01012 * wheel_msf}" iyz="${-4.64239E-08 * wheel_msf}" izz="${0.01012 * wheel_msf}" />
+				<inertia
+					ixx="${0.01875 * wheel_msf}"
+					ixy="${0 * wheel_msf}"
+					ixz="${0 * wheel_msf}"
+					iyy="${0.01012 * wheel_msf}"
+					iyz="${0 * wheel_msf}"
+					izz="${0 * wheel_msf}" />
 			</inertial>
 			<visual>
 				<origin xyz="0 0 0" rpy="0 0 0" />
 				<geometry>
-					<mesh filename="package://propbot_description/meshes/propbot_wheel.STL" />>
+					<mesh filename="package://propbot_description/meshes/propbot_wheel.STL" />
 				</geometry>
 				<material name="wheel_material">
@@ -41,5 +46,5 @@
 			</visual>
 			<collision>
-				<origin xyz="0 0 0" rpy="${M_PI/2} 0 0" />
+				<origin xyz="0 0 0" rpy="0 0 0" />
 				<geometry>
 					<cylinder length="${wheel_length}" radius="${wheel_radius}" />
