Commit message: Enable Realsense, make better mounting position

File: vehicle_autonomy/propbot_description/urdf/propbot.urdf.xacro (robot description, xacro)
@@ -123,15 +123,15 @@
     </joint>
   </xacro:if>
-  <xacro:if value="$(arg kinect_enabled)">
-    <xacro:sensor_arch prefix="" parent="top_plate_link">
-      <origin xyz="-0.35 0 0.51" rpy="0 0 -3.14"/>
-    </xacro:sensor_arch>
-    <joint name="kinect_frame_joint" type="fixed">
-      <origin xyz="$(arg kinect_xyz)" rpy="$(arg kinect_rpy)" />
-      <parent link="sensor_arch_mount_link"/>
-      <child link="camera_link"/>
-    </joint>
-    <xacro:kinect_camera prefix="camera" robot_namespace="$(arg robot_namespace)"/>
-  </xacro:if>
+  <xacro:sensor_arch prefix="" parent="top_plate_link">
+    <origin xyz="-0.35 0 0.51" rpy="0 0 -3.14"/>
+  </xacro:sensor_arch>
+  <link name="camera_link"/>
+  <joint name="kinect_frame_joint" type="fixed">
+    <origin xyz="$(arg kinect_xyz)" rpy="$(arg kinect_rpy)" />
+    <parent link="sensor_arch_mount_link"/>
+    <child link="camera_link"/>
+  </joint>
+  <gazebo reference="camera_link">
+  </gazebo>
   <gazebo>
     <plugin name="gazebo_ros_control" filename="libgazebo_ros_control.so">

Commit message: Add realsense mounting configuration (Disabled)

File: vehicle_autonomy/propbot_description/urdf/propbot.urdf.xacro (robot description, xacro)
@@ -123,4 +123,16 @@
     </joint>
   </xacro:if>
+  <xacro:if value="$(arg kinect_enabled)">
+    <xacro:sensor_arch prefix="" parent="top_plate_link">
+      <origin xyz="-0.35 0 0.51" rpy="0 0 -3.14"/>
+    </xacro:sensor_arch>
+    <joint name="kinect_frame_joint" type="fixed">
+      <origin xyz="$(arg kinect_xyz)" rpy="$(arg kinect_rpy)" />
+      <parent link="sensor_arch_mount_link"/>
+      <child link="camera_link"/>
+    </joint>
+    <xacro:kinect_camera prefix="camera" robot_namespace="$(arg robot_namespace)"/>
+  </xacro:if>
+  <!-- Realsense Mounting (Currently Unused)
   <xacro:sensor_arch prefix="" parent="top_plate_link">
     <origin xyz="-0.35 0 0.51" rpy="0 0 -3.14"/>
@@ -134,4 +146,5 @@
   <gazebo reference="camera_link">
   </gazebo>
+  -->
   <gazebo>
     <plugin name="gazebo_ros_control" filename="libgazebo_ros_control.so">

Commit message: added realsense urdf

File: vehicle_autonomy/propbot_description/urdf/propbot.urdf.xacro (robot description, xacro)
@@ -133,5 +133,7 @@
       <child link="camera_link"/>
     </joint>
-    <xacro:kinect_camera prefix="camera" robot_namespace="$(arg robot_namespace)"/>
+    <realsense_d435 name="camera" parent="sensor_arch_mount_link">
+      <origin xyz="$(arg depth_camera_xyz)" rpy="$(arg depth_camera_rpy)" robot_namespace="$(arg robot_namespace)"/>
+     </realsense_d435>
   </xacro:if>
   <!-- TODO: Enable Realsense -->

Commit message: Removed commented sections

File: vehicle_autonomy/propbot_description/urdf/propbot.urdf.xacro (robot description, xacro)
@@ -137,18 +137,4 @@
      </realsense_d435>
   </xacro:if>
-  <!-- TODO: Enable Realsense -->
-  <!-- Realsense Mounting
-  <xacro:sensor_arch prefix="" parent="top_plate_link">
-    <origin xyz="-0.35 0 0.51" rpy="0 0 -3.14"/>
-  </xacro:sensor_arch>
-  <link name="camera_link"/>
-  <joint name="kinect_frame_joint" type="fixed">
-    <origin xyz="$(arg kinect_xyz)" rpy="$(arg kinect_rpy)" />
-    <parent link="sensor_arch_mount_link"/>
-    <child link="camera_link"/>
-  </joint>
-  <gazebo reference="camera_link">
-  </gazebo>
-  -->
   <gazebo>
     <plugin name="gazebo_ros_control" filename="libgazebo_ros_control.so">

Commit message: renamed launch parameters, and adjusted the realsense gazebo parameters to mimic realsense specs (FOV, resolution)

File: vehicle_autonomy/propbot_description/urdf/propbot.urdf.xacro (robot description, xacro)
@@ -25,7 +25,7 @@
   <xacro:arg name="laser_xyz" default="$(optenv PROPBOT_VLP-16_XYZ 0.2206 0.0 0.00635)" />
   <xacro:arg name="laser_rpy" default="$(optenv PROPBOT_VLP-16_RPY 0.0 0.0 0.0)" />
-  <xacro:arg name="kinect_enabled" default="false" />
-  <xacro:arg name="kinect_xyz" default="$(optenv PROPBOT_KINECT_XYZ 0 0 0)" />
-  <xacro:arg name="kinect_rpy" default="$(optenv PROPBOT_KINECT_RPY 0 0.18 3.14)" />
+  <xacro:arg name="rgbd_camera_enabled" default="false" />
+  <xacro:arg name="rgbd_camera_xyz" default="$(optenv PROPBOT_REALSENSE_XYZ 0 0 0)" />
+  <xacro:arg name="rgbd_camera_rpy" default="$(optenv PROPBOT_REALSENSE_RPY 0 0.18 3.14)" />
   <xacro:property name="propbot_front_bumper_extend" value="$(optenv PROPBOT_FRONT_BUMPER_EXTEND 0)" />
   <xacro:property name="propbot_rear_bumper_extend" value="$(optenv PROPBOT_REAR_BUMPER_EXTEND 0)" />
@@ -124,5 +124,5 @@
     </joint>
   </xacro:if>
-  <xacro:if value="$(arg kinect_enabled)">
+  <xacro:if value="$(arg rgbd_camera_enabled)">
     <xacro:sensor_arch prefix="" parent="top_plate_link">
       <origin xyz="-0.35 0 0.51" rpy="0 0 -3.14"/>
@@ -134,5 +134,5 @@
     </joint>
     <realsense_d435 name="camera" parent="sensor_arch_mount_link">
-      <origin xyz="$(arg depth_camera_xyz)" rpy="$(arg depth_camera_rpy)" robot_namespace="$(arg robot_namespace)"/>
+      <origin xyz="$(arg rgbd_camera_xyz)" rpy="$(arg rgbd_camera_rpy)" robot_namespace="$(arg robot_namespace)"/>
      </realsense_d435>
   </xacro:if>

Commit message: updated wheel positions

File: vehicle_autonomy/propbot_description/urdf/propbot.urdf.xacro (robot description, xacro)
@@ -47,5 +47,4 @@
   <!-- Wheel Mounting Positions -->
   <xacro:property name="wheel_to_wheel" value="0.400" /> <!-- distance between wheel axles -->
-  <xacro:property name="center_to_middle_wheel" value="0.400" /> <!-- x distance from origin to middle wheel center -->
   <xacro:property name="track" value="0.9198" /> <!-- y wheel distance, wheel central point to central point -->
   <xacro:property name="wheel_vertical_offset" value="${wheel_radius}" /> <!-- axle to ground distance -->
@@ -103,20 +102,20 @@
   <!-- Propbot wheel macros -->
   <xacro:propbot_wheel wheel_prefix="front_left">
-    <origin xyz="${wheel_to_wheel + center_to_middle_wheel} ${track/2} ${wheel_vertical_offset}" rpy="0 0 0" />
+    <origin xyz="${wheel_to_wheel} ${track/2} ${wheel_vertical_offset}" rpy="0 0 0" />
   </xacro:propbot_wheel>
   <xacro:propbot_wheel wheel_prefix="front_right">
-    <origin xyz="${wheel_to_wheel + center_to_middle_wheel} ${-track/2} ${wheel_vertical_offset}" rpy="0 0 0" />
+    <origin xyz="${wheel_to_wheel} ${-track/2} ${wheel_vertical_offset}" rpy="0 0 0" />
   </xacro:propbot_wheel>
   <xacro:propbot_wheel wheel_prefix="middle_left">
-    <origin xyz="${center_to_middle_wheel} ${track/2} ${wheel_vertical_offset}" rpy="0 0 0" />
+    <origin xyz="0 ${track/2} ${wheel_vertical_offset}" rpy="0 0 0" />
   </xacro:propbot_wheel>
   <xacro:propbot_wheel wheel_prefix="middle_right">
-    <origin xyz="${center_to_middle_wheel} ${-track/2} ${wheel_vertical_offset}" rpy="0 0 0" />
+    <origin xyz="0 ${-track/2} ${wheel_vertical_offset}" rpy="0 0 0" />
   </xacro:propbot_wheel>
   <xacro:propbot_wheel wheel_prefix="rear_left">
-    <origin xyz="${center_to_middle_wheel - wheel_to_wheel} ${track/2} ${wheel_vertical_offset}" rpy="0 0 0" />
+    <origin xyz="${-wheel_to_wheel} ${track/2} ${wheel_vertical_offset}" rpy="0 0 0" />
   </xacro:propbot_wheel>
   <xacro:propbot_wheel wheel_prefix="rear_right">
-    <origin xyz="${center_to_middle_wheel - wheel_to_wheel} ${-track/2} ${wheel_vertical_offset}" rpy="0 0 0" />
+    <origin xyz="${-wheel_to_wheel} ${-track/2} ${wheel_vertical_offset}" rpy="0 0 0" />
   </xacro:propbot_wheel>
   <xacro:propbot_decorate />

Commit message: Final wheel positions. Need to re-add top_plate for sensors

File: vehicle_autonomy/propbot_description/urdf/propbot.urdf.xacro (robot description, xacro)
@@ -50,4 +50,5 @@
   <xacro:property name="track" value="0.9198" /> <!-- y wheel distance, wheel central point to central point -->
   <xacro:property name="wheel_vertical_offset" value="${wheel_radius}" /> <!-- axle to ground distance -->
+  <xacro:property name="wheel_central_offset" value="0.0533" /> <!-- offset from the center -->
   <!-- Base Size -->
   <xacro:property name="base_x_size" value="0.9820" /> <!-- x is front to back -->
@@ -109,20 +110,20 @@
   <!-- Propbot wheel macros -->
   <xacro:propbot_wheel wheel_prefix="front_left">
-    <origin xyz="${track/2} ${wheel_to_wheel + wheel_radius/4 + 0.011} ${wheel_vertical_offset}" rpy="0 ${M_PI} 0" />
+    <origin xyz="${track/2} ${wheel_to_wheel + wheel_central_offset} ${wheel_vertical_offset}" rpy="0 ${M_PI} 0" />
   </xacro:propbot_wheel>
   <xacro:propbot_wheel wheel_prefix="front_right">
-    <origin xyz="${-track/2} ${wheel_to_wheel} ${wheel_vertical_offset}" rpy="0 0 0" />
+    <origin xyz="${-track/2} ${wheel_to_wheel + wheel_central_offset} ${wheel_vertical_offset}" rpy="0 0 0" />
   </xacro:propbot_wheel>
   <xacro:propbot_wheel wheel_prefix="middle_left">
-    <origin xyz="${track/2} 0 ${wheel_vertical_offset}" rpy="0 ${M_PI} 0" />
+    <origin xyz="${track/2} ${wheel_central_offset} ${wheel_vertical_offset}" rpy="0 ${M_PI} 0" />
   </xacro:propbot_wheel>
   <xacro:propbot_wheel wheel_prefix="middle_right">
-    <origin xyz="${-track/2} 0 ${wheel_vertical_offset}" rpy="0 0 0" />
+    <origin xyz="${-track/2} ${wheel_central_offset} ${wheel_vertical_offset}" rpy="0 0 0" />
   </xacro:propbot_wheel>
   <xacro:propbot_wheel wheel_prefix="rear_left">
-    <origin xyz="${track/2} ${-wheel_to_wheel} ${wheel_vertical_offset}" rpy="0 ${M_PI} 0" />
+    <origin xyz="${track/2} ${-wheel_to_wheel + wheel_central_offset} ${wheel_vertical_offset}" rpy="0 ${M_PI} 0" />
   </xacro:propbot_wheel>
   <xacro:propbot_wheel wheel_prefix="rear_right">
-    <origin xyz="${-track/2} ${-wheel_to_wheel} ${wheel_vertical_offset}" rpy="0 0 0" />
+    <origin xyz="${-track/2} ${-wheel_to_wheel + wheel_central_offset} ${wheel_vertical_offset}" rpy="0 0 0" />
   </xacro:propbot_wheel>
   <xacro:propbot_decorate />

Commit message: Added invisible top plate for sensor linking

File: vehicle_autonomy/propbot_description/urdf/propbot.urdf.xacro (robot description, xacro)
@@ -2,5 +2,5 @@
 <!--
 Software License Agreement (BSD)
-\file      propbot-model.urdf.xacro
+\file      propbot.urdf.xacro
 \authors   Paul Bovbel <pbovbel@clearpathrobotics.com>, Devon Ash <dash@clearpathrobotics.com>
 \copyright Copyright (c) 2015, Clearpath Robotics, Inc., All rights reserved.
@@ -55,4 +55,7 @@
   <xacro:property name="base_y_size" value="0.8278" /> <!-- y is side to side -->
   <xacro:property name="base_z_size" value="0.1369" /> <!-- height of the bottom battery plate from the ground -->
+  <!-- Sensor Mounting Values -->
+  <xacro:property name="top_plate_height" value="${0.24845 + wheel_radius}" /> <!-- height from the ground to the top plate-->
+  <xacro:property name="top_plate_front" value="${base_x_size/2}" /> <!-- distance from the origin to the front of the robot-->
   <!-- Base link is the center of the robot's bottom plate -->
   <link name="base_link">
@@ -138,5 +141,5 @@
   <xacro:if value="$(arg rgbd_camera_enabled)">
     <xacro:sensor_arch prefix="" parent="top_plate_link">
-      <origin xyz="-0.35 0 0.51" rpy="0 0 -3.14"/>
+      <origin xyz="0 0 0" rpy="0 0 -${M_PI}"/>
     </xacro:sensor_arch>
     <realsense_d435 name="camera" parent="sensor_arch_mount_link">

Commit message: Fixes to wheel names, addition of passive wheel

File: vehicle_autonomy/propbot_description/urdf/propbot.urdf.xacro (robot description, xacro)
@@ -28,5 +28,5 @@
 <robot name="propbot" xmlns:xacro="http://ros.org/wiki/xacro">
   <xacro:arg name="laser_enabled" default="false" />
-  <xacro:arg name="laser_xyz" default="$(optenv PROPBOT_VLP-16_XYZ 0.2206 0.0 0.00635)" />
+  <xacro:arg name="laser_xyz" default="$(optenv PROPBOT_VLP-16_XYZ 0.2206 0.0 1.4)" />
   <xacro:arg name="laser_rpy" default="$(optenv PROPBOT_VLP-16_RPY 0.0 0.0 0.0)" />
   <xacro:arg name="rgbd_camera_enabled" default="false" />
@@ -39,4 +39,5 @@
   <xacro:include filename="$(find propbot_description)/urdf/decorations.urdf.xacro" />
   <xacro:include filename="$(find propbot_description)/urdf/wheel.urdf.xacro" />
+  <xacro:include filename="$(find propbot_description)/urdf/passive_wheel.urdf.xacro" />
   <xacro:include filename="$(find propbot_description)/urdf/accessories/realsense_d435.urdf.xacro"/>
   <xacro:include filename="$(find propbot_description)/urdf/accessories/sensor_arch.urdf.xacro"/>
@@ -45,4 +46,5 @@
   <xacro:property name="M_PI" value="3.14159"/>
   <!-- Wheel Properties -->
+  <xacro:property name="wheel_length" value="0.08975" />
   <xacro:property name="wheel_radius" value="0.127" />
   <!-- Wheel Mounting Positions -->
@@ -112,20 +114,20 @@
   </gazebo>
   <!-- Propbot wheel macros -->
-  <xacro:propbot_wheel wheel_prefix="front_left">
+  <xacro:propbot_wheel wheel_prefix="front_right">
     <origin xyz="${track/2} ${wheel_to_wheel + wheel_central_offset} ${wheel_vertical_offset}" rpy="0 ${M_PI} 0" />
   </xacro:propbot_wheel>
-  <xacro:propbot_wheel wheel_prefix="front_right">
+  <xacro:propbot_wheel wheel_prefix="front_left">
     <origin xyz="${-track/2} ${wheel_to_wheel + wheel_central_offset} ${wheel_vertical_offset}" rpy="0 0 0" />
   </xacro:propbot_wheel>
-  <xacro:propbot_wheel wheel_prefix="middle_left">
+  <xacro:propbot_passive_wheel wheel_prefix="middle_right">
     <origin xyz="${track/2} ${wheel_central_offset} ${wheel_vertical_offset}" rpy="0 ${M_PI} 0" />
-  </xacro:propbot_wheel>
-  <xacro:propbot_wheel wheel_prefix="middle_right">
+  </xacro:propbot_passive_wheel>
+  <xacro:propbot_passive_wheel wheel_prefix="middle_left">
     <origin xyz="${-track/2} ${wheel_central_offset} ${wheel_vertical_offset}" rpy="0 0 0" />
+  </xacro:propbot_passive_wheel>
+  <xacro:propbot_wheel wheel_prefix="rear_right">
+    <origin xyz="${track/2} ${-wheel_to_wheel + wheel_central_offset} ${wheel_vertical_offset}" rpy="0 ${M_PI} 0" />
   </xacro:propbot_wheel>
   <xacro:propbot_wheel wheel_prefix="rear_left">
-    <origin xyz="${track/2} ${-wheel_to_wheel + wheel_central_offset} ${wheel_vertical_offset}" rpy="0 ${M_PI} 0" />
-  </xacro:propbot_wheel>
-  <xacro:propbot_wheel wheel_prefix="rear_right">
     <origin xyz="${-track/2} ${-wheel_to_wheel + wheel_central_offset} ${wheel_vertical_offset}" rpy="0 0 0" />
   </xacro:propbot_wheel>

Commit message: Adjusted origin and introduction of mass and inertial scaling

File: vehicle_autonomy/propbot_description/urdf/propbot.urdf.xacro (robot description, xacro)
@@ -45,4 +45,9 @@
   <!-- Define Constant(s) -->
   <xacro:property name="M_PI" value="3.14159"/>
+  <!-- Inertia and Mass Scaling -->
+  <xacro:property name="robot_mass" value="82"/>          <!-- Approximate robot mass is approx 82kg, SolidWorks model incorrect -->
+  <xacro:property name="wheel_mass" value="2.96542"/>     <!-- Wheel mass as reported by SW -->
+  <xacro:property name="chassis_mass" value="19.52246"/>  <!-- Chassis mass as reported by SW -->
+  <xacro:property name="msf" value="${robot_mass/(chassis_mass + 6*wheel_mass)}"/> <!-- Mass scale factor: use to scale masses and inertial values -->
   <!-- Wheel Properties -->
   <xacro:property name="wheel_length" value="0.08975" />
@@ -69,5 +74,5 @@
     </visual>
     <collision>
-      <origin xyz="0 0 ${base_z_size/4}" rpy="0 0 0" />
+      <origin xyz="0 ${wheel_central_offset} ${base_z_size/4}" rpy="0 0 0" />
       <geometry>
         <box size="${base_x_size} ${base_y_size} ${base_z_size/2}"/>
@@ -75,5 +80,5 @@
     </collision>
     <collision>
-      <origin xyz="0 0 ${base_z_size*3/4-0.01}" rpy="0 0 0" />
+      <origin xyz="0 ${wheel_central_offset} ${base_z_size*3/4-0.01}" rpy="0 0 0" />
       <geometry>
         <box size="${base_x_size*4/5} ${base_y_size} ${base_z_size/2-0.02}"/>
@@ -93,7 +98,8 @@
   <link name="inertial_link">
     <inertial>
-      <mass value="19.52246" />
+      <mass value="${chassis_mass*msf}"/>
       <origin xyz="-0.004962 0.106799 0.42243" />
-      <inertia ixx="0.42226" ixy="0.00028" ixz="-0.00012" iyy="0.46973" iyz="0.000170" izz="0.16238" />
+      <inertia ixx="${0.42226*msf}" ixy="${0.00028*msf}" ixz="${-0.00012*msf}"
+               iyy="${0.46973*msf}" iyz="${0.00017*msf}" izz="${0.16238*msf}" />
     </inertial>
   </link>
@@ -115,20 +121,20 @@
   <!-- Propbot wheel macros -->
   <xacro:propbot_wheel wheel_prefix="front_right">
-    <origin xyz="${track/2} ${wheel_to_wheel + wheel_central_offset} ${wheel_vertical_offset}" rpy="0 ${M_PI} 0" />
+    <origin xyz="${track/2} ${wheel_to_wheel} ${wheel_vertical_offset}" rpy="0 ${M_PI} 0" />
   </xacro:propbot_wheel>
   <xacro:propbot_wheel wheel_prefix="front_left">
-    <origin xyz="${-track/2} ${wheel_to_wheel + wheel_central_offset} ${wheel_vertical_offset}" rpy="0 0 0" />
+    <origin xyz="${-track/2} ${wheel_to_wheel} ${wheel_vertical_offset}" rpy="0 0 0" />
   </xacro:propbot_wheel>
   <xacro:propbot_passive_wheel wheel_prefix="middle_right">
-    <origin xyz="${track/2} ${wheel_central_offset} ${wheel_vertical_offset}" rpy="0 ${M_PI} 0" />
+    <origin xyz="${track/2} 0 ${wheel_vertical_offset}" rpy="0 ${M_PI} 0" />
   </xacro:propbot_passive_wheel>
   <xacro:propbot_passive_wheel wheel_prefix="middle_left">
-    <origin xyz="${-track/2} ${wheel_central_offset} ${wheel_vertical_offset}" rpy="0 0 0" />
+    <origin xyz="${-track/2} 0 ${wheel_vertical_offset}" rpy="0 0 0" />
   </xacro:propbot_passive_wheel>
   <xacro:propbot_wheel wheel_prefix="rear_right">
-    <origin xyz="${track/2} ${-wheel_to_wheel + wheel_central_offset} ${wheel_vertical_offset}" rpy="0 ${M_PI} 0" />
+    <origin xyz="${track/2} ${-wheel_to_wheel} ${wheel_vertical_offset}" rpy="0 ${M_PI} 0" />
   </xacro:propbot_wheel>
   <xacro:propbot_wheel wheel_prefix="rear_left">
-    <origin xyz="${-track/2} ${-wheel_to_wheel + wheel_central_offset} ${wheel_vertical_offset}" rpy="0 0 0" />
+    <origin xyz="${-track/2} ${-wheel_to_wheel} ${wheel_vertical_offset}" rpy="0 0 0" />
   </xacro:propbot_wheel>
   <xacro:propbot_decorate />

Commit message: Adjusted origin and introduction of mass and inertial scaling?

File: vehicle_autonomy/propbot_description/urdf/propbot.urdf.xacro (robot description, xacro)
@@ -45,4 +45,9 @@
   <!-- Define Constant(s) -->
   <xacro:property name="M_PI" value="3.14159"/>
+  <!-- Inertia and Mass Scaling -->
+  <xacro:property name="robot_mass" value="82"/>          <!-- Approximate robot mass is approx 82kg, SolidWorks model incorrect -->
+  <xacro:property name="wheel_mass" value="2.96542"/>     <!-- Wheel mass as reported by SW -->
+  <xacro:property name="chassis_mass" value="19.52246"/>  <!-- Chassis mass as reported by SW -->
+  <xacro:property name="msf" value="${robot_mass/(chassis_mass + 6*wheel_mass)}"/> <!-- Mass scale factor: use to scale masses and inertial values -->
   <!-- Wheel Properties -->
   <xacro:property name="wheel_length" value="0.08975" />
@@ -69,5 +74,5 @@
     </visual>
     <collision>
-      <origin xyz="0 0 ${base_z_size/4}" rpy="0 0 0" />
+      <origin xyz="0 ${wheel_central_offset} ${base_z_size/4}" rpy="0 0 0" />
       <geometry>
         <box size="${base_x_size} ${base_y_size} ${base_z_size/2}"/>
@@ -75,5 +80,5 @@
     </collision>
     <collision>
-      <origin xyz="0 0 ${base_z_size*3/4-0.01}" rpy="0 0 0" />
+      <origin xyz="0 ${wheel_central_offset} ${base_z_size*3/4-0.01}" rpy="0 0 0" />
       <geometry>
         <box size="${base_x_size*4/5} ${base_y_size} ${base_z_size/2-0.02}"/>
@@ -93,7 +98,8 @@
   <link name="inertial_link">
     <inertial>
-      <mass value="19.52246" />
+      <mass value="${chassis_mass*msf}"/>
       <origin xyz="-0.004962 0.106799 0.42243" />
-      <inertia ixx="0.42226" ixy="0.00028" ixz="-0.00012" iyy="0.46973" iyz="0.000170" izz="0.16238" />
+      <inertia ixx="${0.42226*msf}" ixy="${0.00028*msf}" ixz="${-0.00012*msf}"
+               iyy="${0.46973*msf}" iyz="${0.00017*msf}" izz="${0.16238*msf}" />
     </inertial>
   </link>
@@ -115,20 +121,20 @@
   <!-- Propbot wheel macros -->
   <xacro:propbot_wheel wheel_prefix="front_right">
-    <origin xyz="${track/2} ${wheel_to_wheel + wheel_central_offset} ${wheel_vertical_offset}" rpy="0 ${M_PI} 0" />
+    <origin xyz="${track/2} ${wheel_to_wheel} ${wheel_vertical_offset}" rpy="0 ${M_PI} 0" />
   </xacro:propbot_wheel>
   <xacro:propbot_wheel wheel_prefix="front_left">
-    <origin xyz="${-track/2} ${wheel_to_wheel + wheel_central_offset} ${wheel_vertical_offset}" rpy="0 0 0" />
+    <origin xyz="${-track/2} ${wheel_to_wheel} ${wheel_vertical_offset}" rpy="0 0 0" />
   </xacro:propbot_wheel>
   <xacro:propbot_passive_wheel wheel_prefix="middle_right">
-    <origin xyz="${track/2} ${wheel_central_offset} ${wheel_vertical_offset}" rpy="0 ${M_PI} 0" />
+    <origin xyz="${track/2} 0 ${wheel_vertical_offset}" rpy="0 ${M_PI} 0" />
   </xacro:propbot_passive_wheel>
   <xacro:propbot_passive_wheel wheel_prefix="middle_left">
-    <origin xyz="${-track/2} ${wheel_central_offset} ${wheel_vertical_offset}" rpy="0 0 0" />
+    <origin xyz="${-track/2} 0 ${wheel_vertical_offset}" rpy="0 0 0" />
   </xacro:propbot_passive_wheel>
   <xacro:propbot_wheel wheel_prefix="rear_right">
-    <origin xyz="${track/2} ${-wheel_to_wheel + wheel_central_offset} ${wheel_vertical_offset}" rpy="0 ${M_PI} 0" />
+    <origin xyz="${track/2} ${-wheel_to_wheel} ${wheel_vertical_offset}" rpy="0 ${M_PI} 0" />
   </xacro:propbot_wheel>
   <xacro:propbot_wheel wheel_prefix="rear_left">
-    <origin xyz="${-track/2} ${-wheel_to_wheel + wheel_central_offset} ${wheel_vertical_offset}" rpy="0 0 0" />
+    <origin xyz="${-track/2} ${-wheel_to_wheel} ${wheel_vertical_offset}" rpy="0 0 0" />
   </xacro:propbot_wheel>
   <xacro:propbot_decorate />

File: vehicle_autonomy/propbot_description/urdf/wheel.urdf.xacro (robot description, xacro)
@@ -26,7 +26,8 @@
 			<!-- Following values extracted from URDF exported from Solidworks -->
 			<inertial>
-				<mass value="2.96542" />
+				<mass value="${wheel_mass*msf}" />
 				<origin xyz="0 0 0" />
-				<inertia  ixx="0.01875" ixy="1.054410E-15" ixz="6.83081E-07" iyy="0.01012" iyz="-4.64239E-08" izz="0.01012" />
+				<inertia  ixx="${0.01875*msf}" ixy="${1.054410E-15*msf}" ixz="${6.83081E-07*msf}"
+				          iyy="${0.01012*msf}" iyz="${-4.64239E-08*msf}" izz="${0.01012*msf}" />
 			</inertial>
 			<visual>
