Commit message: Updated .rviz files to update link set, modified base_link origin

File: vehicle_autonomy/propbot_description/urdf/propbot.urdf.xacro (robot description, xacro)
@@ -28,5 +28,5 @@
 <robot name="propbot" xmlns:xacro="http://ros.org/wiki/xacro">
   <xacro:arg name="laser_enabled" default="false" />
-  <xacro:arg name="laser_xyz" default="$(optenv PROPBOT_VLP-16_XYZ 0.2206 0.0 1.4)" />
+  <xacro:arg name="laser_xyz" default="$(optenv PROPBOT_VLP-16_XYZ 0.2206 0.0 0)" />
   <xacro:arg name="laser_rpy" default="$(optenv PROPBOT_VLP-16_RPY 0.0 0.0 0.0)" />
   <xacro:arg name="rgbd_camera_enabled" default="false" />
@@ -63,6 +63,6 @@
   <xacro:property name="base_z_size" value="0.1369" /> <!-- height of the bottom battery plate from the ground -->
   <!-- Sensor Mounting Values -->
-  <xacro:property name="top_plate_height" value="${0.24845 + wheel_radius}" /> <!-- height from the ground to the top plate-->
-  <xacro:property name="top_plate_front" value="${base_x_size/2}" /> <!-- distance from the origin to the front of the robot-->
+  <xacro:property name="top_plate_height" value="${0.24845 + wheel_radius}" /> <!-- height from the ground to the top plate -->
+  <xacro:property name="top_plate_front" value="${base_x_size/2}" /> <!-- distance from the origin to the front of the robot -->
   <!-- Base link is the center of the robot's bottom plate -->
   <link name="base_link">
@@ -74,5 +74,5 @@
     </visual>
     <collision>
-      <origin xyz="0 ${wheel_central_offset} ${base_z_size/4}" rpy="0 0 0" />
+      <origin xyz="0 ${wheel_central_offset + wheel_length/2} ${base_z_size/4}" rpy="0 0 0" />
       <geometry>
         <box size="${base_x_size} ${base_y_size} ${base_z_size/2}"/>
@@ -80,5 +80,5 @@
     </collision>
     <collision>
-      <origin xyz="0 ${wheel_central_offset} ${base_z_size*3/4-0.01}" rpy="0 0 0" />
+      <origin xyz="0 ${wheel_central_offset + wheel_length/2} ${base_z_size*3/4-0.01}" rpy="0 0 0" />
       <geometry>
         <box size="${base_x_size*4/5} ${base_y_size} ${base_z_size/2-0.02}"/>

Commit message: Fixes inertia issues

File: vehicle_autonomy/propbot_description/urdf/propbot.urdf.xacro (robot description, xacro)
@@ -48,7 +48,11 @@
   <xacro:property name="robot_mass" value="82"/>          <!-- Approximate robot mass is approx 82kg, SolidWorks model incorrect -->
   <xacro:property name="wheel_mass" value="2.96542"/>     <!-- Wheel mass as reported by SW -->
-  <xacro:property name="chassis_mass" value="19.52246"/>  <!-- Chassis mass as reported by SW -->
-  <xacro:property name="msf" value="${robot_mass/(chassis_mass + 6*wheel_mass)}"/>  <!-- Mass scale factor: use to scale masses and inertial values -->
-  <!-- <xacro:property name="msf" value="1"/> Mass scale factor: use to scale masses and inertial values -->
+  <!-- <xacro:property name="chassis_mass" value="19.52246"/>   -->
+  <!-- Chassis mass as reported by SW -->
+  <xacro:property name="chassis_mass" value="70.00"/>
+  <!-- <xacro:property name="msf" value="${robot_mass/(chassis_mass + 6*wheel_mass)}"/>   -->
+  <!-- Mass scale factor: use to scale masses and inertial values -->
+  <xacro:property name="msf" value="1"/>
+  <!-- Mass scale factor: use to scale masses and inertial values -->
   <!-- Wheel Properties -->
   <xacro:property name="wheel_length" value="0.08975" />
@@ -123,11 +127,11 @@
   </xacro:propbot_wheel>
   <xacro:propbot_wheel wheel_prefix="rear_left">
-    <origin xyz="${-track/2 + wheel_radius/2} ${wheel_to_wheel} ${wheel_vertical_offset}" rpy="0 0 ${-M_PI/2}" />
+    <origin xyz="${-track/2 + (2/3)*wheel_radius} ${wheel_to_wheel} ${wheel_vertical_offset}" rpy="0 0 ${-M_PI/2}" />
   </xacro:propbot_wheel>
   <xacro:propbot_passive_wheel wheel_prefix="left">
-    <origin xyz="0 ${wheel_to_wheel} ${wheel_vertical_offset}" rpy="0 0 ${-M_PI/2}" />
+    <origin xyz="${wheel_radius/3} ${wheel_to_wheel} ${wheel_vertical_offset}" rpy="0 0 ${-M_PI/2}" />
   </xacro:propbot_passive_wheel>
   <xacro:propbot_passive_wheel wheel_prefix="right">
-    <origin xyz="0 ${-wheel_to_wheel} ${wheel_vertical_offset}" rpy="0 0 ${-M_PI/2}" />
+    <origin xyz="${wheel_radius/3} ${-wheel_to_wheel} ${wheel_vertical_offset}" rpy="0 0 ${-M_PI/2}" />
   </xacro:propbot_passive_wheel>
   <xacro:propbot_wheel wheel_prefix="front_right">
@@ -135,5 +139,5 @@
   </xacro:propbot_wheel>
   <xacro:propbot_wheel wheel_prefix="rear_right">
-    <origin xyz="${-track/2 + wheel_radius/2} ${-wheel_to_wheel} ${wheel_vertical_offset}" rpy="0 0 ${-M_PI/2}" />
+    <origin xyz="${-track/2 + (2/3)*wheel_radius} ${-wheel_to_wheel} ${wheel_vertical_offset}" rpy="0 0 ${-M_PI/2}" />
   </xacro:propbot_wheel>
   <xacro:propbot_decorate />

Commit message: Fixed camera stand and realsense mounting

File: vehicle_autonomy/propbot_description/urdf/propbot.urdf.xacro (robot description, xacro)
@@ -58,6 +58,6 @@
   <xacro:arg name="laser_rpy" default="$(optenv PROPBOT_VLP-16_RPY 0 0 0)" />
   <xacro:arg name="rgbd_camera_enabled" default="false" />
-  <xacro:arg name="rgbd_camera_xyz" default="$(optenv PROPBOT_REALSENSE_XYZ 0 0 0.95)" />
-  <xacro:arg name="rgbd_camera_rpy" default="$(optenv PROPBOT_REALSENSE_RPY 0 0.18 3.14)" />
+  <xacro:arg name="rgbd_camera_xyz" default="$(optenv PROPBOT_REALSENSE_XYZ 0 0 0)" />
+  <xacro:arg name="rgbd_camera_rpy" default="$(optenv PROPBOT_REALSENSE_RPY 0 0.18 0)" />
   <!--
   ***********************************************************************************************
@@ -236,5 +236,5 @@
   <xacro:if value="$(arg rgbd_camera_enabled)">
     <xacro:sensor_arch prefix="" parent="top_plate_link">
-      <origin xyz="0 0 0" rpy="0 0 -${M_PI}"/>
+      <origin xyz="${base_x_size/2 - 0.05} ${-base_y_size/2 + 0.035} 0.89" rpy="0 0 0"/>
     </xacro:sensor_arch>
     <realsense_d435 name="camera" parent="sensor_arch_mount_link">

Commit message: Unity mass scale factor

File: vehicle_autonomy/propbot_description/urdf/propbot.urdf.xacro (robot description, xacro)
@@ -98,5 +98,6 @@
   <xacro:property name="chassis_izz" value="0.16238" />
   <!-- Robot frame mass scale factor: use to scale chassis and base link masses and inertial values -->
-  <xacro:property name="frame_msf" value="${robot_mass/chassis_mass}" />
+  <!-- <xacro:property name="frame_msf" value="${robot_mass/chassis_mass}" />   -->
+  <xacro:property name="frame_msf" value="1" />
   <!-- Wheel mass scale factor: use to scale wheel masses and inertial values -->
   <xacro:property name="wheel_msf" value="1" />

Commit message: Scaling wheels and chassis by same factor

File: vehicle_autonomy/propbot_description/urdf/propbot.urdf.xacro (robot description, xacro)
@@ -99,7 +99,7 @@
   <!-- Robot frame mass scale factor: use to scale chassis and base link masses and inertial values -->
   <!-- <xacro:property name="frame_msf" value="${robot_mass/chassis_mass}" />   -->
-  <xacro:property name="frame_msf" value="1" />
+  <xacro:property name="frame_msf" value="${robot_mass/chassis_mass}" />
   <!-- Wheel mass scale factor: use to scale wheel masses and inertial values -->
-  <xacro:property name="wheel_msf" value="1" />
+  <xacro:property name="wheel_msf" value="${robot_mass/chassis_mass}" />
   <!--
   ***********************************************************************************************

Commit message: Reverted back to OG scaling, changed position of middle wheels

File: vehicle_autonomy/propbot_description/urdf/propbot.urdf.xacro (robot description, xacro)
@@ -98,8 +98,7 @@
   <xacro:property name="chassis_izz" value="0.16238" />
   <!-- Robot frame mass scale factor: use to scale chassis and base link masses and inertial values -->
-  <!-- <xacro:property name="frame_msf" value="${robot_mass/chassis_mass}" />   -->
   <xacro:property name="frame_msf" value="${robot_mass/chassis_mass}" />
   <!-- Wheel mass scale factor: use to scale wheel masses and inertial values -->
-  <xacro:property name="wheel_msf" value="${robot_mass/chassis_mass}" />
+  <xacro:property name="wheel_msf" value="${1}" />
   <!--
   ***********************************************************************************************
@@ -216,8 +215,8 @@
   <!-- Middle (passives) -->
   <xacro:propbot_passive_wheel wheel_prefix="left">
-    <origin xyz="${wheel_radius/3} ${wheel_to_wheel} ${wheel_vertical_offset}" rpy="0 0 ${-M_PI/2}" />
+    <origin xyz="0 ${wheel_to_wheel} ${wheel_vertical_offset}" rpy="0 0 ${-M_PI/2}" />
   </xacro:propbot_passive_wheel>
   <xacro:propbot_passive_wheel wheel_prefix="right">
-    <origin xyz="${wheel_radius/3} ${-wheel_to_wheel} ${wheel_vertical_offset}" rpy="0 0 ${-M_PI/2}" />
+    <origin xyz="0 ${-wheel_to_wheel} ${wheel_vertical_offset}" rpy="0 0 ${-M_PI/2}" />
   </xacro:propbot_passive_wheel>
   <!-- Decorate the robot -->

Commit message: removed passive wheels

File: vehicle_autonomy/propbot_description/urdf/propbot.urdf.xacro (robot description, xacro)
@@ -214,10 +214,10 @@
   </xacro:propbot_wheel>
   <!-- Middle (passives) -->
-  <xacro:propbot_passive_wheel wheel_prefix="left">
-    <origin xyz="0 ${wheel_to_wheel} ${wheel_vertical_offset}" rpy="0 0 ${-M_PI/2}" />
+  <!-- <xacro:propbot_passive_wheel wheel_prefix="left">
+    <origin xyz="${wheel_radius/3} ${wheel_to_wheel} ${wheel_vertical_offset}" rpy="0 0 ${-M_PI/2}" />
   </xacro:propbot_passive_wheel>
   <xacro:propbot_passive_wheel wheel_prefix="right">
-    <origin xyz="0 ${-wheel_to_wheel} ${wheel_vertical_offset}" rpy="0 0 ${-M_PI/2}" />
-  </xacro:propbot_passive_wheel>
+    <origin xyz="${wheel_radius/3} ${-wheel_to_wheel} ${wheel_vertical_offset}" rpy="0 0 ${-M_PI/2}" />
+  </xacro:propbot_passive_wheel> -->
   <!-- Decorate the robot -->
   <xacro:propbot_decorate />

Commit message: Centered passive wheels

File: vehicle_autonomy/propbot_description/urdf/propbot.urdf.xacro (robot description, xacro)
@@ -215,8 +215,8 @@
   <!-- Middle (passives) -->
   <xacro:propbot_passive_wheel wheel_prefix="left">
-    <origin xyz="${wheel_radius/3} ${wheel_to_wheel} ${wheel_vertical_offset}" rpy="0 0 ${-M_PI/2}" />
+    <origin xyz="0 ${wheel_to_wheel} ${wheel_vertical_offset}" rpy="0 0 ${-M_PI/2}" />
   </xacro:propbot_passive_wheel>
   <xacro:propbot_passive_wheel wheel_prefix="right">
-    <origin xyz="${wheel_radius/3} ${-wheel_to_wheel} ${wheel_vertical_offset}" rpy="0 0 ${-M_PI/2}" />
+    <origin xyz="0 ${-wheel_to_wheel} ${wheel_vertical_offset}" rpy="0 0 ${-M_PI/2}" />
   </xacro:propbot_passive_wheel>
   <!-- Decorate the robot -->

Commit message: Moved middle wheels towards center

File: vehicle_autonomy/propbot_description/urdf/propbot.urdf.xacro (robot description, xacro)
@@ -215,8 +215,8 @@
   <!-- Middle (passives) -->
   <xacro:propbot_passive_wheel wheel_prefix="left">
-    <origin xyz="0 ${wheel_to_wheel} ${wheel_vertical_offset}" rpy="0 0 ${-M_PI/2}" />
+    <origin xyz="${wheel_radius/5} ${wheel_to_wheel} ${wheel_vertical_offset}" rpy="0 0 ${-M_PI/2}" />
   </xacro:propbot_passive_wheel>
   <xacro:propbot_passive_wheel wheel_prefix="right">
-    <origin xyz="0 ${-wheel_to_wheel} ${wheel_vertical_offset}" rpy="0 0 ${-M_PI/2}" />
+    <origin xyz="${wheel_radius/5} ${-wheel_to_wheel} ${wheel_vertical_offset}" rpy="0 0 ${-M_PI/2}" />
   </xacro:propbot_passive_wheel>
   <!-- Decorate the robot -->

Commit message: Middle wheels towards front

File: vehicle_autonomy/propbot_description/urdf/propbot.urdf.xacro (robot description, xacro)
@@ -215,8 +215,8 @@
   <!-- Middle (passives) -->
   <xacro:propbot_passive_wheel wheel_prefix="left">
-    <origin xyz="${wheel_radius/5} ${wheel_to_wheel} ${wheel_vertical_offset}" rpy="0 0 ${-M_PI/2}" />
+    <origin xyz="${wheel_radius/4} ${wheel_to_wheel} ${wheel_vertical_offset}" rpy="0 0 ${-M_PI/2}" />
   </xacro:propbot_passive_wheel>
   <xacro:propbot_passive_wheel wheel_prefix="right">
-    <origin xyz="${wheel_radius/5} ${-wheel_to_wheel} ${wheel_vertical_offset}" rpy="0 0 ${-M_PI/2}" />
+    <origin xyz="${wheel_radius/4} ${-wheel_to_wheel} ${wheel_vertical_offset}" rpy="0 0 ${-M_PI/2}" />
   </xacro:propbot_passive_wheel>
   <!-- Decorate the robot -->

Commit message: Moved middle wheels slightly back

File: vehicle_autonomy/propbot_description/urdf/propbot.urdf.xacro (robot description, xacro)
@@ -100,5 +100,5 @@
   <xacro:property name="frame_msf" value="${robot_mass/chassis_mass}" />
   <!-- Wheel mass scale factor: use to scale wheel masses and inertial values -->
-  <xacro:property name="wheel_msf" value="${1}" />
+  <xacro:property name="wheel_msf" value="1" />
   <!--
   ***********************************************************************************************
@@ -215,8 +215,8 @@
   <!-- Middle (passives) -->
   <xacro:propbot_passive_wheel wheel_prefix="left">
-    <origin xyz="${wheel_radius/4} ${wheel_to_wheel} ${wheel_vertical_offset}" rpy="0 0 ${-M_PI/2}" />
+    <origin xyz="0.027 ${wheel_to_wheel} ${wheel_vertical_offset}" rpy="0 0 ${-M_PI/2}" />
   </xacro:propbot_passive_wheel>
   <xacro:propbot_passive_wheel wheel_prefix="right">
-    <origin xyz="${wheel_radius/4} ${-wheel_to_wheel} ${wheel_vertical_offset}" rpy="0 0 ${-M_PI/2}" />
+    <origin xyz="$0.027 ${-wheel_to_wheel} ${wheel_vertical_offset}" rpy="0 0 ${-M_PI/2}" />
   </xacro:propbot_passive_wheel>
   <!-- Decorate the robot -->

Commit message: Fixed typo error

File: vehicle_autonomy/propbot_description/urdf/propbot.urdf.xacro (robot description, xacro)
@@ -218,5 +218,5 @@
   </xacro:propbot_passive_wheel>
   <xacro:propbot_passive_wheel wheel_prefix="right">
-    <origin xyz="$0.027 ${-wheel_to_wheel} ${wheel_vertical_offset}" rpy="0 0 ${-M_PI/2}" />
+    <origin xyz="0.027 ${-wheel_to_wheel} ${wheel_vertical_offset}" rpy="0 0 ${-M_PI/2}" />
   </xacro:propbot_passive_wheel>
   <!-- Decorate the robot -->

Commit message: Moved FL wheel out slightly

File: vehicle_autonomy/propbot_description/urdf/propbot.urdf.xacro (robot description, xacro)
@@ -208,5 +208,5 @@
   <!-- Left -->
   <xacro:propbot_wheel wheel_prefix="front_left">
-    <origin xyz="${track/2} ${wheel_to_wheel} ${wheel_vertical_offset}" rpy="0 0 ${-M_PI/2}" />
+    <origin xyz="${track/2 + 0.1} ${wheel_to_wheel + 0.1} ${wheel_vertical_offset}" rpy="0 0 ${-M_PI/2}" />
   </xacro:propbot_wheel>
   <xacro:propbot_wheel wheel_prefix="rear_left">

Commit message: Moved inertial origin to (0.1, 0.1, z)

File: vehicle_autonomy/propbot_description/urdf/propbot.urdf.xacro (robot description, xacro)
@@ -166,5 +166,5 @@
     <inertial>
       <mass value="${(chassis_mass + base_link_mass) * frame_msf}"/>
-      <origin xyz="0 0 0.42243" rpy = "${-M_PI/2} ${-M_PI/2} 0" />
+      <origin xyz="0.1 0.1 0.42243" rpy = "${-M_PI/2} ${-M_PI/2} 0" />
       <inertia
         ixx="${(base_ixx + chassis_ixx) * frame_msf}"
@@ -208,5 +208,5 @@
   <!-- Left -->
   <xacro:propbot_wheel wheel_prefix="front_left">
-    <origin xyz="${track/2 + 0.1} ${wheel_to_wheel + 0.1} ${wheel_vertical_offset}" rpy="0 0 ${-M_PI/2}" />
+    <origin xyz="${track/2} ${wheel_to_wheel} ${wheel_vertical_offset}" rpy="0 0 ${-M_PI/2}" />
   </xacro:propbot_wheel>
   <xacro:propbot_wheel wheel_prefix="rear_left">

Commit message: mods inertial origin, x=0.027

File: vehicle_autonomy/propbot_description/urdf/propbot.urdf.xacro (robot description, xacro)
@@ -166,5 +166,5 @@
     <inertial>
       <mass value="${(chassis_mass + base_link_mass) * frame_msf}"/>
-      <origin xyz="0.1 0.1 0.42243" rpy = "${-M_PI/2} ${-M_PI/2} 0" />
+      <origin xyz="0.027 0.05 0.42243" rpy = "${-M_PI/2} ${-M_PI/2} 0" />
       <inertia
         ixx="${(base_ixx + chassis_ixx) * frame_msf}"

Commit message: inertial origin y=0.0375

File: vehicle_autonomy/propbot_description/urdf/propbot.urdf.xacro (robot description, xacro)
@@ -166,5 +166,5 @@
     <inertial>
       <mass value="${(chassis_mass + base_link_mass) * frame_msf}"/>
-      <origin xyz="0.027 0.05 0.42243" rpy = "${-M_PI/2} ${-M_PI/2} 0" />
+      <origin xyz="0.027 0.0375 0.42243" rpy = "${-M_PI/2} ${-M_PI/2} 0" />
       <inertia
         ixx="${(base_ixx + chassis_ixx) * frame_msf}"

Commit message: Decreased x and y

File: vehicle_autonomy/propbot_description/urdf/propbot.urdf.xacro (robot description, xacro)
@@ -166,5 +166,5 @@
     <inertial>
       <mass value="${(chassis_mass + base_link_mass) * frame_msf}"/>
-      <origin xyz="0.027 0.0375 0.42243" rpy = "${-M_PI/2} ${-M_PI/2} 0" />
+      <origin xyz="0.025 0.03 0.42243" rpy = "${-M_PI/2} ${-M_PI/2} 0" />
       <inertia
         ixx="${(base_ixx + chassis_ixx) * frame_msf}"

Commit message: Shifted origin towards left?

File: vehicle_autonomy/propbot_description/urdf/propbot.urdf.xacro (robot description, xacro)
@@ -166,5 +166,5 @@
     <inertial>
       <mass value="${(chassis_mass + base_link_mass) * frame_msf}"/>
-      <origin xyz="0.025 0.03 0.42243" rpy = "${-M_PI/2} ${-M_PI/2} 0" />
+      <origin xyz="0.025 0.04 0.42243" rpy = "${-M_PI/2} ${-M_PI/2} 0" />
       <inertia
         ixx="${(base_ixx + chassis_ixx) * frame_msf}"

Commit message: y=0

File: vehicle_autonomy/propbot_description/urdf/propbot.urdf.xacro (robot description, xacro)
@@ -166,5 +166,5 @@
     <inertial>
       <mass value="${(chassis_mass + base_link_mass) * frame_msf}"/>
-      <origin xyz="0.025 0.04 0.42243" rpy = "${-M_PI/2} ${-M_PI/2} 0" />
+      <origin xyz="0.027 0 0.42243" rpy = "${-M_PI/2} ${-M_PI/2} 0" />
       <inertia
         ixx="${(base_ixx + chassis_ixx) * frame_msf}"

Commit message: Shift middle wheels up

File: vehicle_autonomy/propbot_description/urdf/propbot.urdf.xacro (robot description, xacro)
@@ -215,8 +215,8 @@
   <!-- Middle (passives) -->
   <xacro:propbot_passive_wheel wheel_prefix="left">
-    <origin xyz="0.027 ${wheel_to_wheel} ${wheel_vertical_offset}" rpy="0 0 ${-M_PI/2}" />
+    <origin xyz="0.027 ${wheel_to_wheel} ${wheel_vertical_offset + wheel_radius/10}" rpy="0 0 ${-M_PI/2}" />
   </xacro:propbot_passive_wheel>
   <xacro:propbot_passive_wheel wheel_prefix="right">
-    <origin xyz="0.027 ${-wheel_to_wheel} ${wheel_vertical_offset}" rpy="0 0 ${-M_PI/2}" />
+    <origin xyz="0.027 ${-wheel_to_wheel} ${wheel_vertical_offset + wheel_radius/10}" rpy="0 0 ${-M_PI/2}" />
   </xacro:propbot_passive_wheel>
   <!-- Decorate the robot -->

Commit message: Moved wheels slightly outwards

File: vehicle_autonomy/propbot_description/urdf/propbot.urdf.xacro (robot description, xacro)
@@ -201,22 +201,22 @@
   <!-- Right -->
   <xacro:propbot_wheel wheel_prefix="front_right">
-    <origin xyz="${track/2} ${-wheel_to_wheel} ${wheel_vertical_offset}" rpy="0 0 ${-M_PI/2}" />
+    <origin xyz="${track/2} ${-(wheel_to_wheel + wheel_length)} ${wheel_vertical_offset}" rpy="0 0 ${-M_PI/2}" />
   </xacro:propbot_wheel>
   <xacro:propbot_wheel wheel_prefix="rear_right">
-    <origin xyz="${-track/2 + (2/3)*wheel_radius} ${-wheel_to_wheel} ${wheel_vertical_offset}" rpy="0 0 ${-M_PI/2}" />
+    <origin xyz="${-track/2 + (2/3)*wheel_radius} ${-(wheel_to_wheel + wheel_length)} ${wheel_vertical_offset}" rpy="0 0 ${-M_PI/2}" />
   </xacro:propbot_wheel>
   <!-- Left -->
   <xacro:propbot_wheel wheel_prefix="front_left">
-    <origin xyz="${track/2} ${wheel_to_wheel} ${wheel_vertical_offset}" rpy="0 0 ${-M_PI/2}" />
+    <origin xyz="${track/2} ${wheel_to_wheel + wheel_length} ${wheel_vertical_offset}" rpy="0 0 ${-M_PI/2}" />
   </xacro:propbot_wheel>
   <xacro:propbot_wheel wheel_prefix="rear_left">
-    <origin xyz="${-track/2 + (2/3)*wheel_radius} ${wheel_to_wheel} ${wheel_vertical_offset}" rpy="0 0 ${-M_PI/2}" />
+    <origin xyz="${-track/2 + (2/3)*wheel_radius} ${wheel_to_wheel + wheel_length} ${wheel_vertical_offset}" rpy="0 0 ${-M_PI/2}" />
   </xacro:propbot_wheel>
   <!-- Middle (passives) -->
-  <xacro:propbot_passive_wheel wheel_prefix="left">
-    <origin xyz="0.027 ${wheel_to_wheel} ${wheel_vertical_offset + wheel_radius/10}" rpy="0 0 ${-M_PI/2}" />
+  <xacro:propbot_passive_wheel wheel_prefix="middle_left">
+    <origin xyz="0.027 ${wheel_to_wheel + wheel_length} ${wheel_vertical_offset + wheel_radius/10}" rpy="0 0 ${-M_PI/2}" />
   </xacro:propbot_passive_wheel>
-  <xacro:propbot_passive_wheel wheel_prefix="right">
-    <origin xyz="0.027 ${-wheel_to_wheel} ${wheel_vertical_offset + wheel_radius/10}" rpy="0 0 ${-M_PI/2}" />
+  <xacro:propbot_passive_wheel wheel_prefix="middle_right">
+    <origin xyz="0.027 ${-(wheel_to_wheel + wheel_length)} ${wheel_vertical_offset + wheel_radius/10}" rpy="0 0 ${-M_PI/2}" />
   </xacro:propbot_passive_wheel>
   <!-- Decorate the robot -->

Commit message: Moved wheels in

File: vehicle_autonomy/propbot_description/urdf/propbot.urdf.xacro (robot description, xacro)
@@ -201,22 +201,22 @@
   <!-- Right -->
   <xacro:propbot_wheel wheel_prefix="front_right">
-    <origin xyz="${track/2} ${-(wheel_to_wheel + wheel_length)} ${wheel_vertical_offset}" rpy="0 0 ${-M_PI/2}" />
+    <origin xyz="${track/2} ${-(wheel_to_wheel + wheel_length/2)} ${wheel_vertical_offset}" rpy="0 0 ${-M_PI/2}" />
   </xacro:propbot_wheel>
   <xacro:propbot_wheel wheel_prefix="rear_right">
-    <origin xyz="${-track/2 + (2/3)*wheel_radius} ${-(wheel_to_wheel + wheel_length)} ${wheel_vertical_offset}" rpy="0 0 ${-M_PI/2}" />
+    <origin xyz="${-track/2 + (2/3)*wheel_radius} ${-(wheel_to_wheel + wheel_length/2)} ${wheel_vertical_offset}" rpy="0 0 ${-M_PI/2}" />
   </xacro:propbot_wheel>
   <!-- Left -->
   <xacro:propbot_wheel wheel_prefix="front_left">
-    <origin xyz="${track/2} ${wheel_to_wheel + wheel_length} ${wheel_vertical_offset}" rpy="0 0 ${-M_PI/2}" />
+    <origin xyz="${track/2} ${wheel_to_wheel + wheel_length/2} ${wheel_vertical_offset}" rpy="0 0 ${-M_PI/2}" />
   </xacro:propbot_wheel>
   <xacro:propbot_wheel wheel_prefix="rear_left">
-    <origin xyz="${-track/2 + (2/3)*wheel_radius} ${wheel_to_wheel + wheel_length} ${wheel_vertical_offset}" rpy="0 0 ${-M_PI/2}" />
+    <origin xyz="${-track/2 + (2/3)*wheel_radius} ${wheel_to_wheel + wheel_length/2} ${wheel_vertical_offset}" rpy="0 0 ${-M_PI/2}" />
   </xacro:propbot_wheel>
   <!-- Middle (passives) -->
   <xacro:propbot_passive_wheel wheel_prefix="left">
-    <origin xyz="0.027 ${wheel_to_wheel + wheel_length} ${wheel_vertical_offset + wheel_radius/10}" rpy="0 0 ${-M_PI/2}" />
+    <origin xyz="0.027 ${wheel_to_wheel + wheel_length/2} ${wheel_vertical_offset + wheel_radius/10}" rpy="0 0 ${-M_PI/2}" />
   </xacro:propbot_passive_wheel>
   <xacro:propbot_passive_wheel wheel_prefix="right">
-    <origin xyz="0.027 ${-(wheel_to_wheel + wheel_length)} ${wheel_vertical_offset + wheel_radius/10}" rpy="0 0 ${-M_PI/2}" />
+    <origin xyz="0.027 ${-(wheel_to_wheel + wheel_length/2)} ${wheel_vertical_offset + wheel_radius/10}" rpy="0 0 ${-M_PI/2}" />
   </xacro:propbot_passive_wheel>
   <!-- Decorate the robot -->
