Commit message: Moved origin to the right

File: vehicle_autonomy/propbot_description/urdf/propbot.urdf.xacro (robot description, xacro)
@@ -92,5 +92,5 @@
    <!-- Chassis link inertia-->
   <xacro:property name="chassis_ixx" value="0.42226" />
-  <xacro:property name="chassis_ixy" value="0" />
+  <xacro:property name="chassis_ixy" value="0.00028" />
   <xacro:property name="chassis_ixz" value="0" />
   <xacro:property name="chassis_iyy" value="0.46973" />
@@ -166,5 +166,5 @@
     <inertial>
       <mass value="${(chassis_mass + base_link_mass) * frame_msf}"/>
-      <origin xyz="0.027 0.01 0.42243" rpy = "${-M_PI/2} ${-M_PI/2} 0" />
+      <origin xyz="0.027 -0.01 0.42243" rpy = "${-M_PI/2} ${-M_PI/2} 0" />
       <inertia
         ixx="${(base_ixx + chassis_ixx) * frame_msf}"

Commit message: Inertial values to fix the robot along the x-y plane

File: vehicle_autonomy/propbot_description/urdf/propbot.urdf.xacro (robot description, xacro)
@@ -83,5 +83,12 @@
   <xacro:property name="chassis_mass" value="19.52246"/>
   <xacro:property name="wheel_mass" value="2.96542"/>
-  <!-- Base link inertia-->
+  <!-- Base link inertia
+  Ixx = m(y^2 + z^2)
+  Iyy = m(x^2 + z^2)
+  Izz = m(x^2 + y^2)
+  Ixy = Iyx = -mxy
+  Ixz = Izx = -mxz
+  Iyz = Izy = -myz
+  -->
   <xacro:property name="base_ixx" value="0.083320" />
   <xacro:property name="base_ixy" value="0" />
@@ -101,4 +108,6 @@
   <!-- Wheel mass scale factor: use to scale wheel masses and inertial values -->
   <xacro:property name="wheel_msf" value="1" />
+  <!-- Mass of the base link and frame -->
+  <xacro:property name="inertial_mass" value="${(base_link_mass + chassis_mass) * frame_msf}" />
   <!--
   ***********************************************************************************************
@@ -165,13 +174,13 @@
   <link name="inertial_link">
     <inertial>
-      <mass value="${(chassis_mass + base_link_mass) * frame_msf}"/>
-      <origin xyz="0.027 -0.01 0.42243" rpy = "${-M_PI/2} ${-M_PI/2} 0" />
+      <mass value="${inertial_mass}"/>
+      <origin xyz="0 0 ${base_z_size}" rpy = "${-M_PI/2} ${-M_PI/2} 0" />
       <inertia
-        ixx="${(base_ixx + chassis_ixx) * frame_msf}"
-        ixy="${(base_ixy + chassis_ixy) * frame_msf}"
-        ixz="${(base_ixz + chassis_ixz) * frame_msf}"
-        iyy="${(base_iyy + chassis_iyy) * frame_msf}"
-        iyz="${(base_iyz + chassis_iyz) * frame_msf}"
-        izz="${(base_izz + chassis_izz) * frame_msf}" />
+        ixx="${(0 + base_z_size^2) * inertial_mass}"
+        ixy="${-1 * 0 * 0 * inertial_mass}"
+        ixz="${-1 * 0 * base_z_size * inertial_mass}"
+        iyy="${(0 + base_z_size^2) * inertial_mass}"
+        iyz="${-1 * 0  * base_z_size * inertial_mass}"
+        izz="${(0 + 0) * inertial_mass}" />
     </inertial>
   </link>
